Commit message: Added fake hardware for xarm and husky, removed wheel slip in gazebo sim for now, fixed gazebo sim controller launching with jsb, removed joint state pub since repetitive. Tested gazebo and fake hw

File: husky_xarm6_mcr_description/urdf/husky/a200_wheel_macro.urdf.xacro (robot description, xacro)
@@ -23,16 +23,20 @@
         </link>
         <!-- Gazebo simulation settings -->
-        <xacro:if value="${use_gazebo}">
+        <!-- <xacro:if value="${use_gazebo}"> -->
             <!-- Wheel settings -->
-            <gazebo reference="${wheel_prefix}_wheel">
-                <mu1 value="1.0"/> <!-- Vertical friction coefficient -->
-                <mu2 value="0.5"/> <!-- Lateral and longitudinal friction coefficients -->
-                <kp value="100000000000000000000.0" /> <!-- Stiffness coefficient -->
-                <kd value="1.0" /> <!-- Damping coefficient -->
-                <fdir1 value="1 0 0"/> <!-- Direction of the friction/wheel axis -->
-            </gazebo>
+            <!-- <gazebo reference="${wheel_prefix}_wheel"> -->
+            <!-- Vertical friction coefficient -->
+                <!-- <mu1 value="1.0"/>  -->
+                <!-- Lateral and longitudinal friction coefficients -->
+                <!-- <mu2 value="0.5"/>  -->
+                <!-- Stiffness coefficient -->
+                <!-- <kp value="100000000000000000000.0" />  -->
+                <!-- Damping coefficient -->
+                <!-- <kd value="1.0" />  -->
+                <!-- Direction of the friction/wheel axis -->
+                <!-- <fdir1 value="1 0 0"/>  -->
+            <!-- </gazebo> -->
             <!-- Wheel slip plugin (Ignition/Gazebo) -->
-            <gazebo>
-                <!-- Use the installed Ignition plugin library name and fully-qualified system name -->
+            <!-- <gazebo>
                 <plugin filename="libignition-gazebo-wheel-slip-system.so" name="ignition::gazebo::systems::WheelSlip">
                     <wheel link_name="${wheel_prefix}_wheel">
@@ -44,5 +48,5 @@
                 </plugin>
             </gazebo>
-        </xacro:if>
+        </xacro:if> -->
         <!-- Parent joint is handled by the caller -->
         <!-- <joint name="${wheel_prefix}_wheel_joint" type="continuous">

File: husky_xarm6_mcr_description/urdf/husky/husky_ros2_control.xacro (robot description, xacro)
@@ -1,6 +1,5 @@
 <?xml version="1.0"?>
 <robot xmlns:xacro="http://ros.org/wiki/xacro">
-    <xacro:macro name="husky_ros2_control" params="namespace:='' prefix:='' use_gazebo:=true">
-        <!-- Build namespace prefix -->
+    <xacro:macro name="husky_ros2_control" params="namespace:='' prefix:='' use_gazebo:=true use_fake_hardware:=false">
         <xacro:property name="ns_prefix" value="${namespace}/${prefix}"/>
         <xacro:if value="${use_gazebo}">
@@ -9,32 +8,56 @@
                     <plugin>gz_ros2_control/GazeboSimSystem</plugin>
                 </hardware>
-                <joint name="${ns_prefix}front_left_wheel_joint">
-                    <command_interface name="velocity">
-                        <param name="min">-1</param>
-                        <param name="max">1</param>
-                    </command_interface>
-                    <state_interface name="position"/>
-                    <state_interface name="velocity"/>
-                </joint>
-                <joint name="${ns_prefix}rear_left_wheel_joint">
-                    <command_interface name="velocity">
-                    </command_interface>
-                    <state_interface name="position"/>
-                    <state_interface name="velocity"/>
-                </joint>
-                <joint name="${ns_prefix}front_right_wheel_joint">
-                    <command_interface name="velocity">
-                    </command_interface>
-                    <state_interface name="position"/>
-                    <state_interface name="velocity"/>
-                </joint>
-                <joint name="${ns_prefix}rear_right_wheel_joint">
-                    <command_interface name="velocity">
-                    </command_interface>
-                    <state_interface name="position"/>
-                    <state_interface name="velocity"/>
-                </joint>
+                <xacro:husky_system_joints prefix="${ns_prefix}"/>
             </ros2_control>
         </xacro:if>
+        <xacro:unless value="${use_gazebo}">
+            <ros2_control name="a200_hardware" type="system">
+                <hardware>
+                    <xacro:if value="${use_fake_hardware}">
+                        <plugin>mock_components/GenericSystem</plugin>
+                        <param name="calculate_dynamics">true</param>
+                    </xacro:if>
+                    <xacro:unless value="${use_fake_hardware}">
+                        <!-- Replace later with correct plugin -->
+                        <plugin>mock_components/GenericSystem</plugin>
+                    </xacro:unless>
+                </hardware>
+                <xacro:husky_system_joints prefix="${ns_prefix}"/>
+            </ros2_control>
+        </xacro:unless>
+    </xacro:macro>
+    <xacro:macro name="husky_system_joints" params="prefix">
+        <joint name="${prefix}front_left_wheel_joint">
+            <command_interface name="velocity">
+                <param name="min">-1</param>
+                <param name="max">1</param>
+            </command_interface>
+            <state_interface name="position"/>
+            <state_interface name="velocity"/>
+        </joint>
+        <joint name="${prefix}rear_left_wheel_joint">
+            <command_interface name="velocity">
+                <param name="min">-1</param>
+                <param name="max">1</param>
+            </command_interface>
+            <state_interface name="position"/>
+            <state_interface name="velocity"/>
+        </joint>
+        <joint name="${prefix}front_right_wheel_joint">
+            <command_interface name="velocity">
+                <param name="min">-1</param>
+                <param name="max">1</param>
+            </command_interface>
+            <state_interface name="position"/>
+            <state_interface name="velocity"/>
+        </joint>
+        <joint name="${prefix}rear_right_wheel_joint">
+            <command_interface name="velocity">
+                <param name="min">-1</param>
+                <param name="max">1</param>
+            </command_interface>
+            <state_interface name="position"/>
+            <state_interface name="velocity"/>
+        </joint>
     </xacro:macro>
 </robot>

File: husky_xarm6_mcr_description/urdf/husky_xarm6_mcr.urdf.xacro (robot description, xacro)
@@ -3,4 +3,5 @@
     <!-- Arguments -->
     <xacro:arg name="use_gazebo" default="false"/>
+    <xacro:arg name="use_fake_hardware" default="false"/>
     <xacro:arg name="config_file" default="$(find husky_xarm6_mcr_control)/config/controllers.yaml"/>
     <xacro:arg name="manipulator_ns" default="xarm6"/>
@@ -25,7 +26,17 @@
     <!-- ROS2_CONTROL -->
     <xacro:include filename="$(find husky_xarm6_mcr_description)/urdf/husky/husky_ros2_control.xacro"/>
-    <xacro:husky_ros2_control namespace="$(arg platform_ns)" prefix="$(arg platform_prefix)" use_gazebo="$(arg use_gazebo)"/>
+    <xacro:husky_ros2_control
+        namespace="$(arg platform_ns)"
+        prefix="$(arg platform_prefix)"
+        use_gazebo="$(arg use_gazebo)"
+        use_fake_hardware="$(arg use_fake_hardware)"/>
     <xacro:include filename="$(find husky_xarm6_mcr_description)/urdf/xarm6/xarm6_ros2_control.xacro"/>
-    <xacro:xarm6_ros2_control namespace="$(arg manipulator_ns)" prefix="$(arg manipulator_prefix)" use_gazebo="$(arg use_gazebo)" robot_ip="$(arg robot_ip)" report_type="$(arg report_type)"/>
+    <xacro:xarm6_ros2_control
+        namespace="$(arg manipulator_ns)"
+        prefix="$(arg manipulator_prefix)"
+        use_gazebo="$(arg use_gazebo)"
+        use_fake_hardware="$(arg use_fake_hardware)"
+        robot_ip="$(arg robot_ip)"
+        report_type="$(arg report_type)"/>
     <!-- Gazebo plugin for controller manager (only needed once for whole robot) -->
     <xacro:if value="$(arg use_gazebo)">

File: husky_xarm6_mcr_description/urdf/xarm6/xarm6_ros2_control.xacro (robot description, xacro)
@@ -1,5 +1,6 @@
 <?xml version="1.0"?>
 <robot xmlns:xacro="http://ros.org/wiki/xacro">
-    <xacro:macro name="xarm6_ros2_control" params="use_gazebo:=true namespace:='xarm6' prefix:='' velocity_control:='false'
+    <xacro:macro name="xarm6_ros2_control" params="namespace:='xarm6' prefix:=''
+        use_gazebo:='true' use_fake_hardware:='false' velocity_control:='false'
         robot_ip:='192.168.1.205' report_type:='normal' baud_checkset:='true'
         joint1_lower_limit:=${-2.0*pi}  joint1_upper_limit:=${2.0*pi}
@@ -9,125 +10,109 @@
         joint5_lower_limit:=${-1.6929}  joint5_upper_limit:=${pi}
         joint6_lower_limit:=${-2.0*pi}  joint6_upper_limit:=${2.0*pi}
-        ros2_control_plugin:='uf_robot_hardware/UFRobotSystemHardware'
         hard_interface='EffortJointInterface' reduction='100'">
-        <!-- Build namespace prefix -->
         <xacro:property name="ns_prefix" value="${namespace}/${prefix}"/>
-        <!-- Gazebo Simulated Control -->
         <xacro:if value="${use_gazebo}">
             <ros2_control name="${namespace}/gazebo_system" type="system">
-                <!-- Hardware plugin simulates joint physics -->
                 <hardware>
                     <plugin>gz_ros2_control/GazeboSimSystem</plugin>
                 </hardware>
-                <!-- Expose position + velocity commands/states for all 6 joints -->
-                <joint name="${ns_prefix}joint1">
-                    <command_interface name="position"/>
-                    <command_interface name="velocity"/>
-                    <state_interface name="position">
-                        <param name="initial_value">${pi/2}</param>
-                    </state_interface>
-                    <state_interface name="velocity"/>
-                </joint>
-                <joint name="${ns_prefix}joint2">
-                    <command_interface name="position"/>
-                    <command_interface name="velocity"/>
-                    <state_interface name="position">
-                        <param name="initial_value">-${pi/4}</param>
-                    </state_interface>
-                    <state_interface name="velocity"/>
-                </joint>
-                <joint name="${ns_prefix}joint3">
-                    <command_interface name="position"/>
-                    <command_interface name="velocity"/>
-                    <state_interface name="position">
-                        <param name="initial_value">-${pi/4}</param>
-                    </state_interface>
-                    <state_interface name="velocity"/>
-                </joint>
-                <joint name="${ns_prefix}joint4">
-                    <command_interface name="position"/>
-                    <command_interface name="velocity"/>
-                    <state_interface name="position">
-                        <param name="initial_value">0.0</param>
-                    </state_interface>
-                    <state_interface name="velocity"/>
-                </joint>
-                <joint name="${ns_prefix}joint5">
-                    <command_interface name="position"/>
-                    <command_interface name="velocity"/>
-                    <state_interface name="position">
-                        <param name="initial_value">0.0</param>
-                    </state_interface>
-                    <state_interface name="velocity"/>
-                </joint>
-                <joint name="${ns_prefix}joint6">
-                    <command_interface name="position"/>
-                    <command_interface name="velocity"/>
-                    <state_interface name="position">
-                        <param name="initial_value">${pi/2}</param>
-                    </state_interface>
-                    <state_interface name="velocity"/>
-                </joint>
+                <xacro:xarm_control_joints prefix="${ns_prefix}"
+                    j1_l="${joint1_lower_limit}" j1_u="${joint1_upper_limit}"
+                    j2_l="${joint2_lower_limit}" j2_u="${joint2_upper_limit}"
+                    j3_l="${joint3_lower_limit}" j3_u="${joint3_upper_limit}"
+                    j4_l="${joint4_lower_limit}" j4_u="${joint4_upper_limit}"
+                    j5_l="${joint5_lower_limit}" j5_u="${joint5_upper_limit}"
+                    j6_l="${joint6_lower_limit}" j6_u="${joint6_upper_limit}"/>
             </ros2_control>
         </xacro:if>
-        <!-- Real hardware -->
         <xacro:unless value="${use_gazebo}">
-            <ros2_control name="${ns_prefix}${ros2_control_plugin}" type="system">
+            <ros2_control name="${namespace}/xarm_system" type="system">
                 <hardware>
-                    <plugin>${ros2_control_plugin}</plugin>
-                    <param name="robot_ip">${robot_ip}</param>
-                    <param name="report_type">${report_type}</param>
-                    <param name="baud_checkset">${baud_checkset}</param>
+                    <xacro:if value="${use_fake_hardware}">
+                        <plugin>uf_robot_hardware/UFRobotFakeSystemHardware</plugin>
+                        <param name="hw_ns">${namespace}</param>
+                        <param name="prefix">P${prefix}</param>
+                        <param name="dof">6</param>
+                        <param name="robot_type">xarm</param>
+                    </xacro:if>
+                    <xacro:unless value="${use_fake_hardware}">
+                        <plugin>uf_robot_hardware/UFRobotSystemHardware</plugin>
+                        <param name="robot_ip">${robot_ip}</param>
+                        <param name="report_type">${report_type}</param>
+                        <param name="baud_checkset">${baud_checkset}</param>
+                        <param name="hw_ns">${namespace}</param>
+                        <param name="prefix">P${prefix}</param>
+                        <param name="velocity_control">${velocity_control}</param>
+                        <param name="dof">6</param>
+                        <param name="robot_type">xarm</param>
+                        <param name="add_gripper">false</param>
+                        <param name="add_bio_gripper">false</param>
+                    </xacro:unless>
                 </hardware>
-                <joint name="${ns_prefix}joint1">
-                    <command_interface name="position">
-                        <param name="min">${joint1_lower_limit}</param>
-                        <param name="max">${joint1_upper_limit}</param>
-                    </command_interface>
-                    <state_interface name="position"/>
-                    <state_interface name="velocity"/>
-                </joint>
-                <joint name="${ns_prefix}joint2">
-                    <command_interface name="position">
-                        <param name="min">${joint2_lower_limit}</param>
-                        <param name="max">${joint2_upper_limit}</param>
-                    </command_interface>
-                    <state_interface name="position"/>
-                    <state_interface name="velocity"/>
-                </joint>
-                <joint name="${ns_prefix}joint3">
-                    <command_interface name="position">
-                        <param name="min">${joint3_lower_limit}</param>
-                        <param name="max">${joint3_upper_limit}</param>
-                    </command_interface>
-                    <state_interface name="position"/>
-                    <state_interface name="velocity"/>
-                </joint>
-                <joint name="${ns_prefix}joint4">
-                    <command_interface name="position">
-                        <param name="min">${joint4_lower_limit}</param>
-                        <param name="max">${joint4_upper_limit}</param>
-                    </command_interface>
-                    <state_interface name="position"/>
-                    <state_interface name="velocity"/>
-                </joint>
-                <joint name="${ns_prefix}joint5">
-                    <command_interface name="position">
-                        <param name="min">${joint5_lower_limit}</param>
-                        <param name="max">${joint5_upper_limit}</param>
-                    </command_interface>
-                    <state_interface name="position"/>
-                    <state_interface name="velocity"/>
-                </joint>
-                <joint name="${ns_prefix}joint6">
-                    <command_interface name="position">
-                        <param name="min">${joint6_lower_limit}</param>
-                        <param name="max">${joint6_upper_limit}</param>
-                    </command_interface>
-                    <state_interface name="position"/>
-                    <state_interface name="velocity"/>
-                </joint>
+                <xacro:xarm_control_joints prefix="${ns_prefix}"
+                    j1_l="${joint1_lower_limit}" j1_u="${joint1_upper_limit}"
+                    j2_l="${joint2_lower_limit}" j2_u="${joint2_upper_limit}"
+                    j3_l="${joint3_lower_limit}" j3_u="${joint3_upper_limit}"
+                    j4_l="${joint4_lower_limit}" j4_u="${joint4_upper_limit}"
+                    j5_l="${joint5_lower_limit}" j5_u="${joint5_upper_limit}"
+                    j6_l="${joint6_lower_limit}" j6_u="${joint6_upper_limit}"/>
             </ros2_control>
         </xacro:unless>
     </xacro:macro>
+    <xacro:macro name="xarm_control_joints" params="prefix j1_l j1_u j2_l j2_u j3_l j3_u j4_l j4_u j5_l j5_u j6_l j6_u">
+        <joint name="${prefix}joint1">
+            <command_interface name="position">
+                <param name="min">${j1_l}</param>
+                <param name="max">${j1_u}</param>
+            </command_interface>
+            <command_interface name="velocity"/>
+            <state_interface name="position"><param name="initial_value">${pi/2}</param></state_interface>
+            <state_interface name="velocity"/>
+        </joint>
+        <joint name="${prefix}joint2">
+            <command_interface name="position">
+                <param name="min">${j2_l}</param>
+                <param name="max">${j2_u}</param>
+            </command_interface>
+            <command_interface name="velocity"/>
+            <state_interface name="position"><param name="initial_value">-${pi/4}</param></state_interface>
+            <state_interface name="velocity"/>
+        </joint>
+        <joint name="${prefix}joint3">
+            <command_interface name="position">
+                <param name="min">${j3_l}</param>
+                <param name="max">${j3_u}</param>
+            </command_interface>
+            <command_interface name="velocity"/>
+            <state_interface name="position"><param name="initial_value">-${pi/4}</param></state_interface>
+            <state_interface name="velocity"/>
+        </joint>
+        <joint name="${prefix}joint4">
+            <command_interface name="position">
+                <param name="min">${j4_l}</param>
+                <param name="max">${j4_u}</param>
+            </command_interface>
+            <command_interface name="velocity"/>
+            <state_interface name="position"><param name="initial_value">0.0</param></state_interface>
+            <state_interface name="velocity"/>
+        </joint>
+        <joint name="${prefix}joint5">
+            <command_interface name="position">
+                <param name="min">${j5_l}</param>
+                <param name="max">${j5_u}</param>
+            </command_interface>
+            <command_interface name="velocity"/>
+            <state_interface name="position"><param name="initial_value">0.0</param></state_interface>
+            <state_interface name="velocity"/>
+        </joint>
+        <joint name="${prefix}joint6">
+            <command_interface name="position">
+                <param name="min">${j6_l}</param>
+                <param name="max">${j6_u}</param>
+            </command_interface>
+            <command_interface name="velocity"/>
+            <state_interface name="position"><param name="initial_value">${pi/2}</param></state_interface>
+            <state_interface name="velocity"/>
+        </joint>
+    </xacro:macro>
 </robot>
