Commit message: Gazebo ignition working changed mesh file path in xacro

File: husky_xarm6_mcr_description/urdf/husky/a200_macro.urdf.xacro (robot description, xacro)
@@ -19,5 +19,6 @@
         <origin xyz="0 0 0" rpy="0 0 0" />
         <geometry>
-          <mesh filename="package://clearpath_platform_description/meshes/a200/base_link.dae" />
+          <mesh filename="file://$(find clearpath_platform_description)/meshes/a200/base_link.dae" />
+          <!-- <mesh filename="package://clearpath_platform_description/meshes/a200/base_link.dae" /> -->
         </geometry>
       </visual>
@@ -47,5 +48,6 @@
         <origin xyz="0 0 0" rpy="0 0 0" />
         <geometry>
-          <mesh filename="package://clearpath_platform_description/meshes/a200/top_chassis.dae" />
+          <mesh filename="file://$(find clearpath_platform_description)/meshes/a200/top_chassis.dae" />
+          <!-- <mesh filename="package://clearpath_platform_description/meshes/a200/top_chassis.dae" /> -->
         </geometry>
       </visual>

File: husky_xarm6_mcr_description/urdf/husky/a200_wheel_macro.urdf.xacro (robot description, xacro)
@@ -11,5 +11,6 @@
         <origin xyz="0 0 0" rpy="0 0 0" />
         <geometry>
-          <mesh filename="package://clearpath_platform_description/meshes/a200/wheel.dae" />
+          <!-- <mesh filename="package://clearpath_platform_description/meshes/a200/wheel.dae" /> -->
+          <mesh filename="file://$(find clearpath_platform_description)/meshes/a200/wheel.dae" />
         </geometry>
       </visual>

File: husky_xarm6_mcr_description/urdf/risers/x_rail_macro.urdf.xacro (robot description, xacro)
@@ -8,5 +8,6 @@
                 <origin xyz="0 0 0" rpy="0 0 0"/>
                 <geometry>
-                    <mesh filename="package://husky_xarm6_mcr_description/meshes/x_rail_riser.dae" scale="1 1 1"/>
+                    <!-- <mesh filename="package://husky_xarm6_mcr_description/meshes/x_rail_riser.dae" scale="1 1 1"/> -->
+                    <mesh filename="file://$(find husky_xarm6_mcr_description)/meshes/x_rail_riser.dae"/>
                 </geometry>
             </visual>
@@ -14,5 +15,6 @@
                 <origin xyz="0 0 0" rpy="0 0 0"/>
                 <geometry>
-                    <mesh filename="package://husky_xarm6_mcr_description/meshes/x_rail_riser_collision.stl" scale="1 1 1"/>
+                    <!-- <mesh filename="package://husky_xarm6_mcr_description/meshes/x_rail_riser_collision.stl" scale="1 1 1"/> -->
+                    <mesh filename="file://$(find husky_xarm6_mcr_description)/meshes/x_rail_riser_collision.stl"/>
                 </geometry>
             </collision>
