Commit message: cleaned up xacro files, added gazebo params and settings to the xacro files. Moved slip into the wheel xacro. Passing use_gazebo param throughout.

File: husky_xarm6_mcr_description/urdf/husky/a200_macro.urdf.xacro (robot description, xacro)
@@ -1,226 +1,145 @@
 <?xml version="1.0"?>
 <robot xmlns:xacro="http://ros.org/wiki/xacro">
-  <xacro:property name="M_PI" value="3.14159"/>
-  <xacro:macro name="a200" params="prefix:=''">
-    <!-- Base Size -->
-    <xacro:property name="base_x_size" value="0.98740000" />
-    <xacro:property name="base_y_size" value="0.57090000" />
-    <xacro:property name="base_z_size" value="0.24750000" />
-    <!-- Wheel Mounting Positions -->
-    <xacro:property name="wheelbase" value="0.5120" />
-    <xacro:property name="track" value="0.555" />
-    <xacro:property name="wheel_vertical_offset" value="0.03282" />
-    <!-- Wheel Properties -->
-    <xacro:property name="wheel_length" value="0.1143" />
-    <xacro:property name="wheel_radius" value="0.1651" />
-    <!-- Base link is the center of the robot's bottom plate -->
-    <link name="${prefix}base_link">
-      <visual>
-        <origin xyz="0 0 0" rpy="0 0 0" />
-        <geometry>
-          <mesh filename="file://$(find clearpath_platform_description)/meshes/a200/base_link.dae" />
-          <!-- <mesh filename="package://clearpath_platform_description/meshes/a200/base_link.dae" /> -->
-        </geometry>
-      </visual>
-      <collision>
-        <origin xyz="0 0 ${base_z_size/4}" rpy="0 0 0" />
-        <geometry>
-          <box size="${base_x_size} ${base_y_size} ${base_z_size/2}"/>
-        </geometry>
-      </collision>
-      <collision>
-        <origin xyz="0 0 ${base_z_size*3/4-0.01}" rpy="0 0 0" />
-        <geometry>
-          <box size="${base_x_size*4/5} ${base_y_size} ${base_z_size/2-0.02}"/>
-        </geometry>
-      </collision>
-    </link>
-    <!-- Base footprint is on the ground under the robot -->
-    <link name="${prefix}base_footprint"/>
-    <joint name="${prefix}base_footprint_joint" type="fixed">
-      <origin xyz="0 0 ${wheel_vertical_offset - wheel_radius}" rpy="0 0 0" />
-      <parent link="${prefix}base_link" />
-      <child link="${prefix}base_footprint" />
-    </joint>
-    <!-- Spawn A200 chassis -->
-    <link name="${prefix}top_chassis_link">
-      <visual>
-        <origin xyz="0 0 0" rpy="0 0 0" />
-        <geometry>
-          <mesh filename="file://$(find clearpath_platform_description)/meshes/a200/top_chassis.dae" />
-          <!-- <mesh filename="package://clearpath_platform_description/meshes/a200/top_chassis.dae" /> -->
-        </geometry>
-      </visual>
-    </link>
-    <!-- Attach chassis to the robot -->
-    <joint name="${prefix}top_chassis_joint" type="fixed">
-      <parent link="${prefix}base_link" />
-      <child link="${prefix}top_chassis_link" />
-    </joint>
-    <!-- Inertial link stores the robot's inertial information -->
-    <link name="${prefix}inertial_link">
-      <inertial>
-        <mass value="46.034" />
-        <origin xyz="-0.00065 -0.085 0.062" />
-        <inertia ixx="0.6022" ixy="-0.02364" ixz="-0.1197" iyy="1.7386" iyz="-0.001544" izz="2.0296" />
-      </inertial>
-    </link>
-    <joint name="${prefix}inertial_joint" type="fixed">
-      <origin xyz="0 0 0" rpy="0 0 0" />
-      <parent link="${prefix}base_link" />
-      <child link="${prefix}inertial_link" />
-    </joint>
-    <!-- A200 wheel macros -->
-    <xacro:include filename="$(find husky_xarm6_mcr_description)/urdf/husky/a200_wheel_macro.urdf.xacro" />
-    <xacro:a200_wheel wheel_prefix="${prefix}front_left">
-      <origin xyz="${wheelbase/2} ${track/2} ${wheel_vertical_offset}" rpy="0 0 0" />
-    </xacro:a200_wheel>
-    <xacro:a200_wheel wheel_prefix="${prefix}front_right">
-      <origin xyz="${wheelbase/2} ${-track/2} ${wheel_vertical_offset}" rpy="0 0 0" />
-    </xacro:a200_wheel>
-    <xacro:a200_wheel wheel_prefix="${prefix}rear_left">
-      <origin xyz="${-wheelbase/2} ${track/2} ${wheel_vertical_offset}" rpy="0 0 0" />
-    </xacro:a200_wheel>
-    <xacro:a200_wheel wheel_prefix="${prefix}rear_right">
-      <origin xyz="${-wheelbase/2} ${-track/2} ${wheel_vertical_offset}" rpy="0 0 0" />
-    </xacro:a200_wheel>
-    <!-- Define wheel joints to use prefixed base_link -->
-    <joint name="${prefix}front_left_wheel_joint" type="continuous">
-    <parent link="${prefix}base_link"/>
-    <child link="${prefix}front_left_wheel"/>
-    <origin xyz="${wheelbase/2} ${track/2} ${wheel_vertical_offset}" rpy="0 0 0" />
-    <axis xyz="0 1 0" rpy="0 0 0" />
-    </joint>
-    <joint name="${prefix}front_right_wheel_joint" type="continuous">
-    <parent link="${prefix}base_link"/>
-    <child link="${prefix}front_right_wheel"/>
-    <origin xyz="${wheelbase/2} ${-track/2} ${wheel_vertical_offset}" rpy="0 0 0" />
-    <axis xyz="0 1 0" rpy="0 0 0" />
-    </joint>
-    <joint name="${prefix}rear_left_wheel_joint" type="continuous">
-    <parent link="${prefix}base_link"/>
-    <child link="${prefix}rear_left_wheel"/>
-    <origin xyz="${-wheelbase/2} ${track/2} ${wheel_vertical_offset}" rpy="0 0 0" />
-    <axis xyz="0 1 0" rpy="0 0 0" />
-    </joint>
-    <joint name="${prefix}rear_right_wheel_joint" type="continuous">
-    <parent link="${prefix}base_link"/>
-    <child link="${prefix}rear_right_wheel"/>
-    <origin xyz="${-wheelbase/2} ${-track/2} ${wheel_vertical_offset}" rpy="0 0 0" />
-    <axis xyz="0 1 0" rpy="0 0 0" />
-    </joint>
-    <!-- <gazebo>
-      <plugin filename="libignition-gazebo-wheel-slip-system.so" name="ignition::gazebo::systems::WheelSlip">
-        <wheel link_name="front_left_wheel">
-          <slip_compliance_lateral>1.0</slip_compliance_lateral>
-          <slip_compliance_longitudinal>1.0</slip_compliance_longitudinal>
-          <wheel_normal_force>113</wheel_normal_force>
-          <wheel_radius>${wheel_radius}</wheel_radius>
-        </wheel>
-        <wheel link_name="front_right_wheel">
-          <slip_compliance_lateral>1.0</slip_compliance_lateral>
-          <slip_compliance_longitudinal>1.0</slip_compliance_longitudinal>
-          <wheel_normal_force>113</wheel_normal_force>
-          <wheel_radius>${wheel_radius}</wheel_radius>
-        </wheel>
-        <wheel link_name="rear_left_wheel">
-          <slip_compliance_lateral>1.0</slip_compliance_lateral>
-          <slip_compliance_longitudinal>1.0</slip_compliance_longitudinal>
-          <wheel_normal_force>113</wheel_normal_force>
-          <wheel_radius>${wheel_radius}</wheel_radius>
-        </wheel>
-        <wheel link_name="rear_right_wheel">
-          <slip_compliance_lateral>1.0</slip_compliance_lateral>
-          <slip_compliance_longitudinal>1.0</slip_compliance_longitudinal>
-          <wheel_normal_force>113</wheel_normal_force>
-          <wheel_radius>${wheel_radius}</wheel_radius>
-        </wheel>
-      </plugin>
-    </gazebo> -->
-    <!-- Front bumper mount -->
-    <link name="${prefix}front_bumper_mount"/>
-    <joint name="${prefix}front_bumper_mount_joint" type="fixed">
-      <origin xyz="0.406 0 0.091" rpy="0 0 0" />
-      <parent link="${prefix}base_link" />
-      <child link="${prefix}front_bumper_mount" />
-    </joint>
-    <!-- Rear bumper mount -->
-    <link name="${prefix}rear_bumper_mount"/>
-    <joint name="${prefix}rear_bumper_mount_joint" type="fixed">
-      <origin xyz="-0.406 0 0.091" rpy="0 0 ${M_PI}" />
-      <parent link="${prefix}base_link" />
-      <child link="${prefix}rear_bumper_mount" />
-    </joint>
-    <!-- Default mount -->
-    <link name="${prefix}default_mount"/>
-    <joint name="${prefix}default_mount_joint" type="fixed">
-      <child link="${prefix}default_mount"/>
-      <parent link="${prefix}base_link"/>
-      <origin xyz="0.0 0.0 0.224"/>
-    </joint>
-    <!-- front & rear bumper -->
-    <!-- <xacro:include filename="$(find clearpath_platform_description)/urdf/a200/attachments/bumper.urdf.xacro"/>
-    <xacro:bumper name="front_bumper"
-                model="default"
-                parent_link="front_bumper_mount">
-        <origin xyz="0 0 0" rpy="0 0 0"/>
-    </xacro:bumper>
-    <xacro:bumper name="rear_bumper"
-                model="default"
-                parent_link="rear_bumper_mount">
-        <origin xyz="0 0 0" rpy="0 0 0"/>
-    </xacro:bumper> -->
-    <!-- Gazebo Controller -->
-    <!-- <xacro:include filename="$(find clearpath_platform_description)/urdf/generic/gazebo.urdf.xacro"/> -->
-    <!-- ROS2 controls -->
-    <!-- <xacro:if value="$(arg use_platform_controllers)">
-      <ros2_control name="a200_hardware" type="system">
-        <hardware>
-          <xacro:if value="$(arg is_sim)">
-            <plugin>ign_ros2_control/IgnitionSystem</plugin>
-          </xacro:if>
-          <xacro:unless value="$(arg is_sim)">
-            <plugin>clearpath_hardware_interfaces/A200Hardware</plugin>
-            <param name="wheel_diameter">0.3302</param>
-            <param name="max_accel">5.0</param>
-            <param name="max_speed">1.0</param>
-            <param name="polling_timeout">0.1</param>
-            <param name="serial_port">$(arg serial_port)</param>
-          </xacro:unless>
-        </hardware>
-        <joint name="${prefix}front_left_wheel_joint">
-          <command_interface name="velocity">
-            <param name="min">-1</param>
-            <param name="max">1</param>
-          </command_interface>
-          <state_interface name="position"/>
-          <state_interface name="velocity"/>
+    <xacro:macro name="a200" params="prefix:='' use_gazebo:=true">
+        <!-- Base Size -->
+        <xacro:property name="base_x_size" value="0.98740000" />
+        <xacro:property name="base_y_size" value="0.57090000" />
+        <xacro:property name="base_z_size" value="0.24750000" />
+        <!-- Wheel Mounting Positions -->
+        <xacro:property name="wheelbase" value="0.5120" />
+        <xacro:property name="track" value="0.555" />
+        <xacro:property name="wheel_vertical_offset" value="0.03282" />
+        <!-- Wheel Properties -->
+        <xacro:property name="wheel_length" value="0.1143" />
+        <xacro:property name="wheel_radius" value="0.1651" />
+        <!-- Base link is the center of the robot's bottom plate -->
+        <link name="${prefix}base_link">
+            <visual>
+                <origin xyz="0 0 0" rpy="0 0 0" />
+                <geometry>
+                    <!-- <mesh filename="package://clearpath_platform_description/meshes/a200/base_link.dae" /> -->
+                    <mesh filename="file://$(find clearpath_platform_description)/meshes/a200/base_link.dae" /> <!-- Use this for Gazebo -->
+                </geometry>
+            </visual>
+            <collision>
+                <origin xyz="0 0 ${base_z_size/4}" rpy="0 0 0" />
+                <geometry>
+                    <box size="${base_x_size} ${base_y_size} ${base_z_size/2}"/>
+                </geometry>
+            </collision>
+            <collision>
+                <origin xyz="0 0 ${base_z_size*3/4-0.01}" rpy="0 0 0" />
+                <geometry>
+                    <box size="${base_x_size*4/5} ${base_y_size} ${base_z_size/2-0.02}"/>
+                </geometry>
+            </collision>
+        </link>
+        <!-- Base footprint is on the ground under the robot -->
+        <link name="${prefix}base_footprint"/>
+        <joint name="${prefix}base_footprint_joint" type="fixed">
+            <origin xyz="0 0 ${wheel_vertical_offset - wheel_radius}" rpy="0 0 0" />
+            <parent link="${prefix}base_link" />
+            <child link="${prefix}base_footprint" />
         </joint>
-        <joint name="${prefix}rear_left_wheel_joint">
-          <command_interface name="velocity">
-            <param name="min">-1</param>
-            <param name="max">1</param>
-          </command_interface>
-          <state_interface name="position"/>
-          <state_interface name="velocity"/>
+        <!-- Spawn A200 chassis -->
+        <link name="${prefix}top_chassis_link">
+            <visual>
+                <origin xyz="0 0 0" rpy="0 0 0" />
+                <geometry>
+                    <!-- <mesh filename="package://clearpath_platform_description/meshes/a200/top_chassis.dae" /> -->
+                    <mesh filename="file://$(find clearpath_platform_description)/meshes/a200/top_chassis.dae" /> <!-- Use this for Gazebo -->
+                </geometry>
+            </visual>
+        </link>
+        <!-- Attach chassis to the robot -->
+        <joint name="${prefix}top_chassis_joint" type="fixed">
+            <parent link="${prefix}base_link" />
+            <child link="${prefix}top_chassis_link" />
         </joint>
-        <joint name="${prefix}front_right_wheel_joint">
-          <command_interface name="velocity">
-            <param name="min">-1</param>
-            <param name="max">1</param>
-          </command_interface>
-          <state_interface name="position"/>
-          <state_interface name="velocity"/>
+        <!-- Inertial link stores the robot's inertial information -->
+        <link name="${prefix}inertial_link">
+            <inertial>
+                <mass value="46.034" />
+                <origin xyz="-0.00065 -0.085 0.062" />
+                <inertia ixx="0.6022" ixy="-0.02364" ixz="-0.1197" iyy="1.7386" iyz="-0.001544" izz="2.0296" />
+            </inertial>
+        </link>
+        <joint name="${prefix}inertial_joint" type="fixed">
+            <origin xyz="0 0 0" rpy="0 0 0" />
+            <parent link="${prefix}base_link" />
+            <child link="${prefix}inertial_link" />
         </joint>
-        <joint name="${prefix}rear_right_wheel_joint">
-          <command_interface name="velocity">
-            <param name="min">-1</param>
-            <param name="max">1</param>
-          </command_interface>
-          <state_interface name="position"/>
-          <state_interface name="velocity"/>
+        <!-- A200 wheel macros -->
+        <xacro:include filename="$(find husky_xarm6_mcr_description)/urdf/husky/a200_wheel_macro.urdf.xacro" />
+        <xacro:a200_wheel wheel_prefix="${prefix}front_left" use_gazebo="${use_gazebo}" wheel_length="${wheel_length}" wheel_radius="${wheel_radius}">
+            <origin xyz="${wheelbase/2} ${track/2} ${wheel_vertical_offset}" rpy="0 0 0" />
+        </xacro:a200_wheel>
+        <xacro:a200_wheel wheel_prefix="${prefix}front_right" use_gazebo="${use_gazebo}" wheel_length="${wheel_length}" wheel_radius="${wheel_radius}">
+            <origin xyz="${wheelbase/2} ${-track/2} ${wheel_vertical_offset}" rpy="0 0 0" />
+        </xacro:a200_wheel>
+        <xacro:a200_wheel wheel_prefix="${prefix}rear_left" use_gazebo="${use_gazebo}" wheel_length="${wheel_length}" wheel_radius="${wheel_radius}">
+            <origin xyz="${-wheelbase/2} ${track/2} ${wheel_vertical_offset}" rpy="0 0 0" />
+        </xacro:a200_wheel>
+        <xacro:a200_wheel wheel_prefix="${prefix}rear_right" use_gazebo="${use_gazebo}" wheel_length="${wheel_length}" wheel_radius="${wheel_radius}">
+            <origin xyz="${-wheelbase/2} ${-track/2} ${wheel_vertical_offset}" rpy="0 0 0" />
+        </xacro:a200_wheel>
+        <!-- Define wheel joints to use prefixed base_link -->
+        <joint name="${prefix}front_left_wheel_joint" type="continuous">
+            <parent link="${prefix}base_link"/>
+            <child link="${prefix}front_left_wheel"/>
+            <origin xyz="${wheelbase/2} ${track/2} ${wheel_vertical_offset}" rpy="0 0 0" />
+            <axis xyz="0 1 0" rpy="0 0 0" />
         </joint>
-      </ros2_control>
-    </xacro:if> -->
-  </xacro:macro>
+        <joint name="${prefix}front_right_wheel_joint" type="continuous">
+            <parent link="${prefix}base_link"/>
+            <child link="${prefix}front_right_wheel"/>
+            <origin xyz="${wheelbase/2} ${-track/2} ${wheel_vertical_offset}" rpy="0 0 0" />
+            <axis xyz="0 1 0" rpy="0 0 0" />
+        </joint>
+        <joint name="${prefix}rear_left_wheel_joint" type="continuous">
+            <parent link="${prefix}base_link"/>
+            <child link="${prefix}rear_left_wheel"/>
+            <origin xyz="${-wheelbase/2} ${track/2} ${wheel_vertical_offset}" rpy="0 0 0" />
+            <axis xyz="0 1 0" rpy="0 0 0" />
+        </joint>
+        <joint name="${prefix}rear_right_wheel_joint" type="continuous">
+            <parent link="${prefix}base_link"/>
+            <child link="${prefix}rear_right_wheel"/>
+            <origin xyz="${-wheelbase/2} ${-track/2} ${wheel_vertical_offset}" rpy="0 0 0" />
+            <axis xyz="0 1 0" rpy="0 0 0" />
+        </joint>
+        <!-- Front bumper mount -->
+        <link name="${prefix}front_bumper_mount"/>
+        <joint name="${prefix}front_bumper_mount_joint" type="fixed">
+            <origin xyz="0.406 0 0.091" rpy="0 0 0" />
+            <parent link="${prefix}base_link" />
+            <child link="${prefix}front_bumper_mount" />
+        </joint>
+        <!-- Rear bumper mount -->
+        <link name="${prefix}rear_bumper_mount"/>
+        <joint name="${prefix}rear_bumper_mount_joint" type="fixed">
+            <origin xyz="-0.406 0 0.091" rpy="0 0 ${pi}" />
+            <parent link="${prefix}base_link" />
+            <child link="${prefix}rear_bumper_mount" />
+        </joint>
+        <!-- Default mount -->
+        <link name="${prefix}default_mount"/>
+        <joint name="${prefix}default_mount_joint" type="fixed">
+            <child link="${prefix}default_mount"/>
+            <parent link="${prefix}base_link"/>
+            <origin xyz="0.0 0.0 0.224"/>
+        </joint>
+        <!-- front & rear bumper -->
+        <!-- <xacro:include filename="$(find clearpath_platform_description)/urdf/a200/attachments/bumper.urdf.xacro"/>
+        <xacro:bumper name="front_bumper"
+                    model="default"
+                    parent_link="front_bumper_mount">
+            <origin xyz="0 0 0" rpy="0 0 0"/>
+        </xacro:bumper>
+        <xacro:bumper name="rear_bumper"
+                    model="default"
+                    parent_link="rear_bumper_mount">
+            <origin xyz="0 0 0" rpy="0 0 0"/>
+        </xacro:bumper> -->
+    </xacro:macro>
 </robot>

File: husky_xarm6_mcr_description/urdf/husky/a200_wheel_macro.urdf.xacro (robot description, xacro)
@@ -1,38 +1,55 @@
 <?xml version="1.0"?>
 <robot xmlns:xacro="http://ros.org/wiki/xacro" name="a200_wheel">
-  <xacro:macro name="a200_wheel" params="wheel_prefix *joint_pose">
-    <link name="${wheel_prefix}_wheel">
-      <inertial>
-        <mass value="2.637" />
-        <origin xyz="0 0 0" />
-        <inertia ixx="0.02467" ixy="0" ixz="0" iyy="0.04411" iyz="0" izz="0.02467" />
-      </inertial>
-      <visual>
-        <origin xyz="0 0 0" rpy="0 0 0" />
-        <geometry>
-          <!-- <mesh filename="package://clearpath_platform_description/meshes/a200/wheel.dae" /> -->
-          <mesh filename="file://$(find clearpath_platform_description)/meshes/a200/wheel.dae" />
-        </geometry>
-      </visual>
-      <collision>
-        <origin xyz="0 0 0" rpy="${M_PI/2} 0 0" />
-        <geometry>
-          <cylinder length="${wheel_length}" radius="${wheel_radius}" />
-        </geometry>
-      </collision>
-    </link>
-    <!-- <gazebo reference="${wheel_prefix}_wheel">
-      <mu1 value="1.0"/>
-      <mu2 value="0.5"/>
-      <kp value="100000000000000000000.0" />
-      <kd value="1.0" />
-      <fdir1 value="1 0 0"/>
-    </gazebo> -->
-    <!-- <joint name="${wheel_prefix}_wheel_joint" type="continuous">
-      <parent link="base_link"/>
-      <child link="${wheel_prefix}_wheel"/>
-      <xacro:insert_block name="joint_pose"/>
-      <axis xyz="0 1 0" rpy="0 0 0" />
-    </joint> -->
-  </xacro:macro>
+    <xacro:macro name="a200_wheel" params="wheel_prefix use_gazebo wheel_length wheel_radius *joint_pose">
+        <link name="${wheel_prefix}_wheel">
+            <inertial>
+                <mass value="2.637" />
+                <origin xyz="0 0 0" />
+                <inertia ixx="0.02467" ixy="0" ixz="0" iyy="0.04411" iyz="0" izz="0.02467" />
+            </inertial>
+            <visual>
+                <origin xyz="0 0 0" rpy="0 0 0" />
+                <geometry>
+                    <!-- <mesh filename="package://clearpath_platform_description/meshes/a200/wheel.dae" /> -->
+                    <mesh filename="file://$(find clearpath_platform_description)/meshes/a200/wheel.dae" /> <!-- Use this for Gazebo -->
+                </geometry>
+            </visual>
+            <collision>
+                <origin xyz="0 0 0" rpy="${pi/2} 0 0" />
+                <geometry>
+                    <cylinder length="${wheel_length}" radius="${wheel_radius}" />
+                </geometry>
+            </collision>
+        </link>
+        <!-- Gazebo simulation settings -->
+        <xacro:if value="${use_gazebo}">
+            <!-- Wheel settings -->
+            <gazebo reference="${wheel_prefix}_wheel">
+                <mu1 value="1.0"/> <!-- Vertical friction coefficient -->
+                <mu2 value="0.5"/> <!-- Lateral and longitudinal friction coefficients -->
+                <kp value="100000000000000000000.0" /> <!-- Stiffness coefficient -->
+                <kd value="1.0" /> <!-- Damping coefficient -->
+                <fdir1 value="1 0 0"/> <!-- Direction of the friction/wheel axis -->
+            </gazebo>
+            <!-- Wheel slip plugin (Ignition/Gazebo) -->
+            <gazebo>
+                <!-- Use the installed Ignition plugin library name and fully-qualified system name -->
+                <plugin filename="libignition-gazebo-wheel-slip-system.so" name="ignition::gazebo::systems::WheelSlip">
+                    <wheel link_name="${wheel_prefix}_wheel">
+                        <slip_compliance_lateral>1.0</slip_compliance_lateral>
+                        <slip_compliance_longitudinal>1.0</slip_compliance_longitudinal>
+                        <wheel_normal_force>113</wheel_normal_force>
+                        <wheel_radius>${wheel_radius}</wheel_radius>
+                    </wheel>
+                </plugin>
+            </gazebo>
+        </xacro:if>
+        <!-- Parent joint is handled by the caller -->
+        <!-- <joint name="${wheel_prefix}_wheel_joint" type="continuous">
+            <parent link="base_link"/>
+            <child link="${wheel_prefix}_wheel"/>
+            <xacro:insert_block name="joint_pose"/>
+            <axis xyz="0 1 0" rpy="0 0 0" />
+        </joint> -->
+    </xacro:macro>
 </robot>
