Commit message: cleaned up xacro files, added gazebo params and settings to the xacro files. Moved slip into the wheel xacro. Passing use_gazebo param throughout.

File: husky_xarm6_mcr_description/urdf/husky/husky_ros2_control.xacro (robot description, xacro)
@@ -1,34 +1,53 @@
 <?xml version="1.0"?>
 <robot xmlns:xacro="http://ros.org/wiki/xacro">
-    <xacro:macro name="husky_ros2_control" params="use_gazebo:=true
-        front_left_wheel_joint:='front_left_wheel_joint'
-        rear_left_wheel_joint:='rear_left_wheel_joint'
-        front_right_wheel_joint:='front_right_wheel_joint'
-        rear_right_wheel_joint:='rear_right_wheel_joint'">
+    <xacro:macro name="husky_ros2_control" params="prefix:='' use_gazebo:=true">
         <xacro:if value="${use_gazebo}">
-            <ros2_control name="GazeboSimSystem" type="system">
+            <ros2_control name="a200_hardware" type="system">
                 <hardware>
-                    <plugin>gz_ros2_control/GazeboSimSystem</plugin>
+                    <!-- Enable ros2_control plugin depending on simulator -->
+                    <xacro:if value="${use_gazebo}">
+                        <plugin>gz_ros2_control/GazeboSimSystem</plugin>
+                    </xacro:if>
+                    <!-- <xacro:unless value="$(arg use_gazebo)">
+                        <plugin>clearpath_hardware_interfaces/A200Hardware</plugin>
+                        <param name="wheel_diameter">0.3302</param>
+                        <param name="max_accel">5.0</param>
+                        <param name="max_speed">1.0</param>
+                        <param name="polling_timeout">0.1</param>
+                        <param name="serial_port">$(arg serial_port)</param>
+                    </xacro:unless> -->
                 </hardware>
                 <!-- Wheels provide velocity command & position/velocity state -->
-                <joint name="${front_left_wheel_joint}">
-                <command_interface name="velocity"/>
-                <state_interface name="position"/>
-                <state_interface name="velocity"/>
+                <joint name="${prefix}front_left_wheel_joint">
+                    <command_interface name="velocity">
+                        <param name="min">-1</param>
+                        <param name="max">1</param>
+                    </command_interface>
+                    <state_interface name="position"/>
+                    <state_interface name="velocity"/>
                 </joint>
-                <joint name="${rear_left_wheel_joint}">
-                <command_interface name="velocity"/>
-                <state_interface name="position"/>
-                <state_interface name="velocity"/>
+                <joint name="${prefix}rear_left_wheel_joint">
+                    <command_interface name="velocity">
+                        <param name="min">-1</param>
+                        <param name="max">1</param>
+                    </command_interface>
+                    <state_interface name="position"/>
+                    <state_interface name="velocity"/>
                 </joint>
-                <joint name="${front_right_wheel_joint}">
-                <command_interface name="velocity"/>
-                <state_interface name="position"/>
-                <state_interface name="velocity"/>
+                <joint name="${prefix}front_right_wheel_joint">
+                    <command_interface name="velocity">
+                        <param name="min">-1</param>
+                        <param name="max">1</param>
+                    </command_interface>
+                    <state_interface name="position"/>
+                    <state_interface name="velocity"/>
                 </joint>
-                <joint name="${rear_right_wheel_joint}">
-                <command_interface name="velocity"/>
-                <state_interface name="position"/>
-                <state_interface name="velocity"/>
+                <joint name="${prefix}rear_right_wheel_joint">
+                    <command_interface name="velocity">
+                        <param name="min">-1</param>
+                        <param name="max">1</param>
+                    </command_interface>
+                    <state_interface name="position"/>
+                    <state_interface name="velocity"/>
                 </joint>
             </ros2_control>

File: husky_xarm6_mcr_description/urdf/husky_xarm6_mcr.urdf.xacro (robot description, xacro)
@@ -5,8 +5,7 @@
     <xacro:arg name="manipulator_prefix" default="xarm6_"/>
     <xacro:arg name="platform_prefix" default="a200_"/>
-    <!-- Parameters -->
     <!-- HUSKY PLATFORM & ATTACHMENTS -->
     <xacro:include filename="$(find husky_xarm6_mcr_description)/urdf/husky/a200_macro.urdf.xacro"/>
-    <xacro:a200 prefix="$(arg platform_prefix)"/>
+    <xacro:a200 prefix="$(arg platform_prefix)" use_gazebo="$(arg sim)"/>
     <!-- X-RAIL RISER -->
     <xacro:include filename="$(find husky_xarm6_mcr_description)/urdf/risers/x_rail_macro.urdf.xacro"/>
@@ -16,11 +15,5 @@
     <!-- ROS2_CONTROL -->
     <xacro:include filename="$(find husky_xarm6_mcr_description)/urdf/husky/husky_ros2_control.xacro"/>
-    <xacro:husky_ros2_control
-        use_gazebo="$(arg sim)"
-        front_left_wheel_joint="$(arg platform_prefix)front_left_wheel_joint"
-        rear_left_wheel_joint="$(arg platform_prefix)rear_left_wheel_joint"
-        front_right_wheel_joint="$(arg platform_prefix)front_right_wheel_joint"
-        rear_right_wheel_joint="$(arg platform_prefix)rear_right_wheel_joint"
-    />
+    <xacro:husky_ros2_control prefix="$(arg platform_prefix)" use_gazebo="$(arg sim)"/>
     <gazebo>
         <plugin filename="gz_ros2_control-system" name="gz_ros2_control::GazeboSimROS2ControlPlugin">

Commit message: fixed timing issue which resulted in diff drive controller not functioning

File: husky_xarm6_mcr_description/urdf/husky/a200_macro.urdf.xacro (robot description, xacro)
@@ -90,4 +90,6 @@
             <origin xyz="${wheelbase/2} ${track/2} ${wheel_vertical_offset}" rpy="0 0 0" />
             <axis xyz="0 1 0" rpy="0 0 0" />
+            <limit effort="10000.0" velocity="100.0"/>
+            <dynamics damping="0.0" friction="0.0"/>
         </joint>
         <joint name="${prefix}front_right_wheel_joint" type="continuous">
@@ -96,4 +98,6 @@
             <origin xyz="${wheelbase/2} ${-track/2} ${wheel_vertical_offset}" rpy="0 0 0" />
             <axis xyz="0 1 0" rpy="0 0 0" />
+            <limit effort="10000.0" velocity="100.0"/>
+            <dynamics damping="0.0" friction="0.0"/>
         </joint>
         <joint name="${prefix}rear_left_wheel_joint" type="continuous">
@@ -102,4 +106,6 @@
             <origin xyz="${-wheelbase/2} ${track/2} ${wheel_vertical_offset}" rpy="0 0 0" />
             <axis xyz="0 1 0" rpy="0 0 0" />
+            <limit effort="10000.0" velocity="100.0"/>
+            <dynamics damping="0.0" friction="0.0"/>
         </joint>
         <joint name="${prefix}rear_right_wheel_joint" type="continuous">
@@ -108,4 +114,6 @@
             <origin xyz="${-wheelbase/2} ${-track/2} ${wheel_vertical_offset}" rpy="0 0 0" />
             <axis xyz="0 1 0" rpy="0 0 0" />
+            <limit effort="10000.0" velocity="100.0"/>
+            <dynamics damping="0.0" friction="0.0"/>
         </joint>
         <!-- Front bumper mount -->

File: husky_xarm6_mcr_description/urdf/husky/husky_ros2_control.xacro (robot description, xacro)
@@ -8,4 +8,10 @@
                     <xacro:if value="${use_gazebo}">
                         <plugin>gz_ros2_control/GazeboSimSystem</plugin>
+                        <param name="velocity_proportional_gain">5.0</param>
+                        <param name="velocity_integral_gain">0.0</param>
+                        <param name="velocity_derivative_gain">0.0</param>
+                        <param name="position_proportional_gain">0.0</param>
+                        <param name="position_integral_gain">0.0</param>
+                        <param name="position_derivative_gain">0.0</param>
                     </xacro:if>
                     <!-- <xacro:unless value="$(arg use_gazebo)">
@@ -21,6 +27,6 @@
                 <joint name="${prefix}front_left_wheel_joint">
                     <command_interface name="velocity">
-                        <param name="min">-1</param>
-                        <param name="max">1</param>
+                        <!-- <param name="min">-1</param>
+                        <param name="max">1</param> -->
                     </command_interface>
                     <state_interface name="position"/>
@@ -29,6 +35,6 @@
                 <joint name="${prefix}rear_left_wheel_joint">
                     <command_interface name="velocity">
-                        <param name="min">-1</param>
-                        <param name="max">1</param>
+                        <!-- <param name="min">-1</param>
+                        <param name="max">1</param> -->
                     </command_interface>
                     <state_interface name="position"/>
@@ -37,6 +43,6 @@
                 <joint name="${prefix}front_right_wheel_joint">
                     <command_interface name="velocity">
-                        <param name="min">-1</param>
-                        <param name="max">1</param>
+                        <!-- <param name="min">-1</param>
+                        <param name="max">1</param> -->
                     </command_interface>
                     <state_interface name="position"/>
@@ -45,6 +51,6 @@
                 <joint name="${prefix}rear_right_wheel_joint">
                     <command_interface name="velocity">
-                        <param name="min">-1</param>
-                        <param name="max">1</param>
+                        <!-- <param name="min">-1</param>
+                        <param name="max">1</param> -->
                     </command_interface>
                     <state_interface name="position"/>

Commit message: Added back husky simulation parameters like max min on wheel velocity and limit enforcement in the diff drive controller. Also updated bridge to expose the cmd vel unstamped topic from GZ to ROS and added z axis spawning offset for the robot.

File: husky_xarm6_mcr_description/urdf/husky/a200_macro.urdf.xacro (robot description, xacro)
@@ -90,6 +90,6 @@
             <origin xyz="${wheelbase/2} ${track/2} ${wheel_vertical_offset}" rpy="0 0 0" />
             <axis xyz="0 1 0" rpy="0 0 0" />
-            <limit effort="10000.0" velocity="100.0"/>
-            <dynamics damping="0.0" friction="0.0"/>
+            <!-- <limit effort="10000.0" velocity="100.0"/>
+            <dynamics damping="0.0" friction="0.0"/> -->
         </joint>
         <joint name="${prefix}front_right_wheel_joint" type="continuous">
@@ -98,6 +98,6 @@
             <origin xyz="${wheelbase/2} ${-track/2} ${wheel_vertical_offset}" rpy="0 0 0" />
             <axis xyz="0 1 0" rpy="0 0 0" />
-            <limit effort="10000.0" velocity="100.0"/>
-            <dynamics damping="0.0" friction="0.0"/>
+            <!-- <limit effort="10000.0" velocity="100.0"/>
+            <dynamics damping="0.0" friction="0.0"/> -->
         </joint>
         <joint name="${prefix}rear_left_wheel_joint" type="continuous">
@@ -106,6 +106,6 @@
             <origin xyz="${-wheelbase/2} ${track/2} ${wheel_vertical_offset}" rpy="0 0 0" />
             <axis xyz="0 1 0" rpy="0 0 0" />
-            <limit effort="10000.0" velocity="100.0"/>
-            <dynamics damping="0.0" friction="0.0"/>
+            <!-- <limit effort="10000.0" velocity="100.0"/>
+            <dynamics damping="0.0" friction="0.0"/> -->
         </joint>
         <joint name="${prefix}rear_right_wheel_joint" type="continuous">
@@ -114,6 +114,6 @@
             <origin xyz="${-wheelbase/2} ${-track/2} ${wheel_vertical_offset}" rpy="0 0 0" />
             <axis xyz="0 1 0" rpy="0 0 0" />
-            <limit effort="10000.0" velocity="100.0"/>
-            <dynamics damping="0.0" friction="0.0"/>
+            <!-- <limit effort="10000.0" velocity="100.0"/>
+            <dynamics damping="0.0" friction="0.0"/> -->
         </joint>
         <!-- Front bumper mount -->

File: husky_xarm6_mcr_description/urdf/husky/husky_ros2_control.xacro (robot description, xacro)
@@ -8,10 +8,10 @@
                     <xacro:if value="${use_gazebo}">
                         <plugin>gz_ros2_control/GazeboSimSystem</plugin>
-                        <param name="velocity_proportional_gain">5.0</param>
+                        <!-- <param name="velocity_proportional_gain">5.0</param>
                         <param name="velocity_integral_gain">0.0</param>
                         <param name="velocity_derivative_gain">0.0</param>
                         <param name="position_proportional_gain">0.0</param>
                         <param name="position_integral_gain">0.0</param>
-                        <param name="position_derivative_gain">0.0</param>
+                        <param name="position_derivative_gain">0.0</param> -->
                     </xacro:if>
                     <!-- <xacro:unless value="$(arg use_gazebo)">
@@ -27,6 +27,6 @@
                 <joint name="${prefix}front_left_wheel_joint">
                     <command_interface name="velocity">
-                        <!-- <param name="min">-1</param>
-                        <param name="max">1</param> -->
+                        <param name="min">-1</param>
+                        <param name="max">1</param>
                     </command_interface>
                     <state_interface name="position"/>
@@ -35,6 +35,6 @@
                 <joint name="${prefix}rear_left_wheel_joint">
                     <command_interface name="velocity">
-                        <!-- <param name="min">-1</param>
-                        <param name="max">1</param> -->
+                        <param name="min">-1</param>
+                        <param name="max">1</param>
                     </command_interface>
                     <state_interface name="position"/>
@@ -43,6 +43,6 @@
                 <joint name="${prefix}front_right_wheel_joint">
                     <command_interface name="velocity">
-                        <!-- <param name="min">-1</param>
-                        <param name="max">1</param> -->
+                        <param name="min">-1</param>
+                        <param name="max">1</param>
                     </command_interface>
                     <state_interface name="position"/>
@@ -51,6 +51,6 @@
                 <joint name="${prefix}rear_right_wheel_joint">
                     <command_interface name="velocity">
-                        <!-- <param name="min">-1</param>
-                        <param name="max">1</param> -->
+                        <param name="min">-1</param>
+                        <param name="max">1</param>
                     </command_interface>
                     <state_interface name="position"/>

Commit message: Added odometry and map to control and robot bringup (had to do minor reconstruction on the urdf file). Added a map frame publisher than publishes the map at the same spot at the odom frame for the time being. Also began implementing the next best view planning package and the volumetric representation for the planning scene.

File: husky_xarm6_mcr_description/urdf/husky/a200_macro.urdf.xacro (robot description, xacro)
@@ -38,7 +38,10 @@
         <link name="${prefix}base_footprint"/>
         <joint name="${prefix}base_footprint_joint" type="fixed">
-            <origin xyz="0 0 ${wheel_vertical_offset - wheel_radius}" rpy="0 0 0" />
+            <!-- <origin xyz="0 0 ${wheel_vertical_offset - wheel_radius}" rpy="0 0 0" />
             <parent link="${prefix}base_link" />
-            <child link="${prefix}base_footprint" />
+            <child link="${prefix}base_footprint" /> -->
+            <origin xyz="0 0 ${wheel_radius - wheel_vertical_offset}" rpy="0 0 0"/>
+            <parent link="${prefix}base_footprint"/>
+            <child link="${prefix}base_link"/>
         </joint>
         <!-- Spawn A200 chassis -->

Commit message: Updated the cad visual and collision model for the xrail riser.

File: husky_xarm6_mcr_description/urdf/husky/a200_macro.urdf.xacro (robot description, xacro)
@@ -6,5 +6,5 @@
         <!-- Base Size -->
         <xacro:property name="base_x_size" value="0.98740000" />
-        <xacro:property name="base_y_size" value="0.57090000" />
+        <xacro:property name="base_y_size" value="0.43" />
         <xacro:property name="base_z_size" value="0.24750000" />
         <!-- Wheel Mounting Positions -->

File: husky_xarm6_mcr_description/urdf/husky_xarm6_mcr.urdf.xacro (robot description, xacro)
@@ -17,10 +17,10 @@
     <xacro:include filename="$(find husky_xarm6_mcr_description)/urdf/risers/x_rail_macro.urdf.xacro"/>
     <xacro:x_rail_riser namespace="$(arg platform_ns)" prefix="$(arg platform_prefix)" parent_link="$(arg platform_ns)/$(arg platform_prefix)default_mount">
-        <origin xyz="0.0 0.0 0.0" rpy="0 0 ${-pi/2}"/>
+        <origin xyz="0.0 0.0 0.02" rpy="0 0 ${-pi/2}"/>
     </xacro:x_rail_riser>
     <!-- XARM6 -->
     <xacro:include filename="$(find husky_xarm6_mcr_description)/urdf/xarm6/xarm6_macro.urdf.xacro"/>
     <xacro:xarm6 namespace="$(arg manipulator_ns)" prefix="$(arg manipulator_prefix)" model_num="1303" parent_link="$(arg platform_ns)/$(arg platform_prefix)x_rail_riser_link">
-        <origin xyz="0.09500000 0 0.31610000" rpy="0 0 0"/>
+        <origin xyz="0.09500000 0 0.33" rpy="0 0 0"/>
     </xacro:xarm6>
     <!-- ROS2_CONTROL -->

File: husky_xarm6_mcr_description/urdf/risers/x_rail_macro.urdf.xacro (robot description, xacro)
@@ -5,20 +5,40 @@
         <!-- Build namespace prefix -->
         <xacro:property name="ns_prefix" value="${namespace}/${prefix}"/>
-        <xacro:property name="height" value="0.33" />
-        <xacro:property name="width" value="0.46" />
-        <xacro:property name="depth" value="1.1" />
+        <!-- Riser Size -->
+        <xacro:property name="riser_x_size" value="0.43" />
+        <xacro:property name="riser_y_extension" value="0.25" />
+        <xacro:property name="riser_y_size" value="0.55" />
+        <xacro:property name="riser_z_size" value="0.28" />
+        <!-- Riser Origin -->
+        <xacro:property name="riser_x_origin" value="0" />
+        <xacro:property name="riser_y_origin" value="-0.078" />
+        <xacro:property name="riser_z_origin" value="0" />
+        <xacro:property name="riser_y_offset" value="0.125" />
+        <xacro:property name="riser_z_offset" value="-0.02" />
+        <!-- Battery Size -->
+        <xacro:property name="battery_z_size" value="0.08" />
+        <xacro:property name="battery_z_origin" value="${0.26 + battery_z_size/2}" />
         <!-- X-Rail Riser Link -->
         <link name="${ns_prefix}x_rail_riser_link">
             <visual>
-                <origin xyz="0 0 0" rpy="0 0 0"/>
+                <origin xyz="${riser_x_origin} ${riser_y_origin} ${riser_z_origin}" rpy="0 0 0"/>
                 <geometry>
                     <!-- <mesh filename="package://husky_xarm6_mcr_description/meshes/x_rail_riser.dae" scale="1 1 1"/> -->
-                    <mesh filename="file://$(find husky_xarm6_mcr_description)/meshes/x_rail_riser.dae"/>
+                    <!-- <mesh filename="file://$(find husky_xarm6_mcr_description)/meshes/x_rail_riser.dae"/> -->
+                    <mesh filename="file://$(find husky_xarm6_mcr_description)/meshes/Platform_Electronics.dae"/>
                 </geometry>
             </visual>
+            <!-- X-rail collisions -->
             <collision>
-                <origin xyz="0 0 ${height/2}" rpy="0 0 0"/>
+                <origin xyz="${riser_x_origin} ${riser_y_offset} ${riser_z_origin + riser_z_offset + riser_z_size/2}" rpy="0 0 0"/>
                 <geometry>
-                    <box size="${width} ${depth} ${height}"/>
+                    <box size="${riser_x_size} ${riser_y_size + riser_y_extension} ${riser_z_size}"/>
+                </geometry>
+            </collision>
+            <!-- Mounted battery collisions -->
+            <collision>
+                <origin xyz="0 0 ${battery_z_origin}" rpy="0 0 0"/>
+                <geometry>
+                    <box size="${riser_x_size} ${riser_y_size} ${battery_z_size}"/>
                 </geometry>
             </collision>
