Commit message: added xarm6 controller. bring up in gazebo sim

File: husky_xarm6_mcr_description/urdf/husky_xarm6_mcr.urdf.xacro (robot description, xacro)
@@ -13,7 +13,14 @@
         <origin xyz="0.0 0.0 0.0" rpy="0 0 ${-pi/2}"/>
     </xacro:x_rail_riser>
+    <!-- XARM6 -->
+    <xacro:include filename="$(find husky_xarm6_mcr_description)/urdf/xarm6/xarm6_macro.urdf.xacro"/>
+    <xacro:xarm6 prefix="$(arg manipulator_prefix)" model_num="1303" parent_link="x_rail_riser_link">
+        <origin xyz="0.09500000 0 0.31610000" rpy="0 0 ${-pi/2}"/>
+    </xacro:xarm6>
     <!-- ROS2_CONTROL -->
     <xacro:include filename="$(find husky_xarm6_mcr_description)/urdf/husky/husky_ros2_control.xacro"/>
     <xacro:husky_ros2_control prefix="$(arg platform_prefix)" use_gazebo="$(arg sim)"/>
+    <xacro:include filename="$(find husky_xarm6_mcr_description)/urdf/xarm6/xarm6_ros2_control.xacro"/>
+    <xacro:xarm6_ros2_control prefix="$(arg manipulator_prefix)" use_gazebo="$(arg sim)"/>
     <gazebo>
         <plugin filename="gz_ros2_control-system" name="gz_ros2_control::GazeboSimROS2ControlPlugin">
@@ -21,9 +28,4 @@
         </plugin>
     </gazebo>
-    <!-- XARM6 -->
-    <!-- <xacro:include filename="$(find husky_xarm6_mcr_description)/urdf/xarm6/xarm6_macro.urdf.xacro"/>
-    <xacro:xarm6 prefix="$(arg manipulator_prefix)" model_num="1303" parent_link="x_rail_riser_link">
-        <origin xyz="0.09500000 0 0.31610000" rpy="0 0 ${-pi/2}"/>
-    </xacro:xarm6> -->
     <!-- MULTI CAMERA RIG -->
     <!-- <xacro:include filename="$(find multi_cam_rig_description)/urdf/multi_cam_rig_macro.urdf.xacro"/>

File: husky_xarm6_mcr_description/urdf/xarm6/xarm6_macro.urdf.xacro (robot description, xacro)
@@ -1,5 +1,5 @@
 <?xml version="1.0"?>
 <robot xmlns:xacro="http://ros.org/wiki/xacro">
-  <xacro:macro name="xarm6" params="prefix
+  <xacro:macro name="xarm6" params="prefix use_gazebo:=true
     joint1_lower_limit:=${-2.0*pi}  joint1_upper_limit:=${2.0*pi}
     joint2_lower_limit:=${-2.059}  joint2_upper_limit:=${2.0944}
@@ -46,6 +46,126 @@
     <xacro:property name="kinematics_config" value="${xacro.load_yaml(kinematics_params_file)}"/>
     <xacro:property name="kinematics_params" value="${kinematics_config['kinematics']}"/>
-    <xacro:property name="mesh_path" value="package://xarm_description/meshes" scope="parent"/>
+    <xacro:property name="mesh_path" value="$(find xarm_description)/meshes" scope="parent"/>
     <xacro:property name="mesh_suffix" value="stl" scope="parent"/>
+    <!-- xarm material colors -->
+    <xacro:include filename="$(find xarm_description)/urdf/common/common.material.xacro" />
+    <xacro:common_material prefix="${prefix}"/>
+    <!-- xarm links -->
+    <link name="${prefix}base_link">
+      <inertial>
+        <origin xyz="0.0 0.0 0.09103" rpy="0 0 0" />
+        <mass value="2.7" />
+        <inertia
+          ixx="0.00494875" ixy="-3.5E-06" ixz="1.25E-05"
+          iyy="0.00494174" iyz="1.67E-06" izz="0.002219" />
+      </inertial>
+      <xacro:common_link_visual
+        mesh_filename="${visual_dir}/link_base"
+        origin_xyz="0 0 0"
+        origin_rpy="0 0 0"
+        material_name="${prefix}White" />
+      <xacro:common_link_collision
+        mesh_filename="${collision_dir}/link_base"
+        add_mesh_suffix="${add_mesh_suffix}"
+        other_mesh_suffix="${collison_mesh_suffix}"
+        origin_xyz="0 0 0"
+        origin_rpy="0 0 0" />
+    </link>
+    <link name="${prefix}link1">
+      <xacro:common_link_inertial
+        link_inertial_params="${inertial_params['link1']}"
+        origin_rpy="0 0 0"/>
+      <xacro:common_link_visual
+        mesh_filename="${visual_dir}/link1"
+        origin_xyz="0 0 0"
+        origin_rpy="0 0 0"
+        material_name="${prefix}White" />
+      <xacro:common_link_collision
+        mesh_filename="${collision_dir}/link1"
+        add_mesh_suffix="${add_mesh_suffix}"
+        other_mesh_suffix="${collison_mesh_suffix}"
+        origin_xyz="0 0 0"
+        origin_rpy="0 0 0" />
+    </link>
+    <link name="${prefix}link2">
+      <xacro:common_link_inertial
+        link_inertial_params="${inertial_params['link2']}"
+        origin_rpy="0 0 0"/>
+      <xacro:common_link_visual
+        mesh_filename="${visual_dir}/link2"
+        origin_xyz="0 0 0"
+        origin_rpy="0 0 0"
+        material_name="${prefix}White" />
+      <xacro:common_link_collision
+        mesh_filename="${collision_dir}/link2"
+        add_mesh_suffix="${add_mesh_suffix}"
+        other_mesh_suffix="${collison_mesh_suffix}"
+        origin_xyz="0 0 0"
+        origin_rpy="0 0 0" />
+    </link>
+    <link name="${prefix}link3">
+      <xacro:common_link_inertial
+        link_inertial_params="${inertial_params['link3']}"
+        origin_rpy="0 0 0"/>
+      <xacro:common_link_visual
+        mesh_filename="${visual_dir}/link3"
+        origin_xyz="0 0 0"
+        origin_rpy="0 0 0"
+        material_name="${prefix}White" />
+      <xacro:common_link_collision
+        mesh_filename="${collision_dir}/link3"
+        add_mesh_suffix="${add_mesh_suffix}"
+        other_mesh_suffix="${collison_mesh_suffix}"
+        origin_xyz="0 0 0"
+        origin_rpy="0 0 0" />
+    </link>
+    <link name="${prefix}link4">
+      <xacro:common_link_inertial
+        link_inertial_params="${inertial_params['link4']}"
+        origin_rpy="0 0 0"/>
+      <xacro:common_link_visual
+        mesh_filename="${visual_dir}/link4"
+        origin_xyz="0 0 0"
+        origin_rpy="0 0 0"
+        material_name="${prefix}White" />
+      <xacro:common_link_collision
+        mesh_filename="${collision_dir}/link4"
+        add_mesh_suffix="${add_mesh_suffix}"
+        other_mesh_suffix="${collison_mesh_suffix}"
+        origin_xyz="0 0 0"
+        origin_rpy="0 0 0" />
+    </link>
+    <link name="${prefix}link5">
+      <xacro:common_link_inertial
+        link_inertial_params="${inertial_params['link5']}"
+        origin_rpy="0 0 0"/>
+      <xacro:common_link_visual
+        mesh_filename="${visual_dir}/link5"
+        origin_xyz="0 0 0"
+        origin_rpy="0 0 0"
+        material_name="${prefix}White" />
+      <xacro:common_link_collision
+        mesh_filename="${collision_dir}/link5"
+        add_mesh_suffix="${add_mesh_suffix}"
+        other_mesh_suffix="${collison_mesh_suffix}"
+        origin_xyz="0 0 0"
+        origin_rpy="0 0 0" />
+    </link>
+    <link name="${prefix}link6">
+      <xacro:common_link_inertial
+        link_inertial_params="${inertial_params['link6']}"
+        origin_rpy="0 0 0"/>
+      <xacro:common_link_visual
+        mesh_filename="${link6_visual}"
+        origin_xyz="0 0 0"
+        origin_rpy="0 0 0"
+        material_name="${prefix}Silver" />
+      <xacro:common_link_collision
+        mesh_filename="${link6_collision}"
+        add_mesh_suffix="${add_mesh_suffix}"
+        other_mesh_suffix="${collison_mesh_suffix}"
+        origin_xyz="0 0 0"
+        origin_rpy="0 0 0" />
+    </link>
     <!-- Optional: attach base link to an external parent link -->
     <xacro:if value="${parent_link != ''}">
@@ -56,44 +176,5 @@
       </joint>
     </xacro:if>
-    <!-- xarm material colors -->
-    <xacro:include filename="$(find xarm_description)/urdf/common/common.material.xacro" />
-    <xacro:common_material prefix="${prefix}"/>
-    <!-- xarm links and joints -->
-    <link name="${prefix}base_link">
-      <inertial>
-        <origin xyz="0.0 0.0 0.09103" rpy="0 0 0" />
-        <mass value="2.7" />
-        <inertia
-          ixx="0.00494875" ixy="-3.5E-06" ixz="1.25E-05"
-          iyy="0.00494174" iyz="1.67E-06" izz="0.002219" />
-      </inertial>
-      <xacro:common_link_visual
-        mesh_filename="${visual_dir}/link_base"
-        origin_xyz="0 0 0"
-        origin_rpy="0 0 0"
-        material_name="${prefix}White" />
-      <xacro:common_link_collision
-        mesh_filename="${collision_dir}/link_base"
-        add_mesh_suffix="${add_mesh_suffix}"
-        other_mesh_suffix="${collison_mesh_suffix}"
-        origin_xyz="0 0 0"
-        origin_rpy="0 0 0" />
-    </link>
-    <link name="${prefix}link1">
-      <xacro:common_link_inertial
-        link_inertial_params="${inertial_params['link1']}"
-        origin_rpy="0 0 0"/>
-      <xacro:common_link_visual
-        mesh_filename="${visual_dir}/link1"
-        origin_xyz="0 0 0"
-        origin_rpy="0 0 0"
-        material_name="${prefix}White" />
-      <xacro:common_link_collision
-        mesh_filename="${collision_dir}/link1"
-        add_mesh_suffix="${add_mesh_suffix}"
-        other_mesh_suffix="${collison_mesh_suffix}"
-        origin_xyz="0 0 0"
-        origin_rpy="0 0 0" />
-    </link>
+    <!-- xarm joints -->
     <joint name="${prefix}joint1" type="revolute">
       <parent link="${prefix}base_link"/>
@@ -109,20 +190,4 @@
       <dynamics damping="1.0" friction="1.0"/>
     </joint>
-    <link name="${prefix}link2">
-      <xacro:common_link_inertial
-        link_inertial_params="${inertial_params['link2']}"
-        origin_rpy="0 0 0"/>
-      <xacro:common_link_visual
-        mesh_filename="${visual_dir}/link2"
-        origin_xyz="0 0 0"
-        origin_rpy="0 0 0"
-        material_name="${prefix}White" />
-      <xacro:common_link_collision
-        mesh_filename="${collision_dir}/link2"
-        add_mesh_suffix="${add_mesh_suffix}"
-        other_mesh_suffix="${collison_mesh_suffix}"
-        origin_xyz="0 0 0"
-        origin_rpy="0 0 0" />
-    </link>
     <joint name="${prefix}joint2" type="revolute">
       <parent link="${prefix}link1"/>
@@ -138,20 +203,4 @@
       <dynamics damping="1.0" friction="1.0"/>
     </joint>
-    <link name="${prefix}link3">
-      <xacro:common_link_inertial
-        link_inertial_params="${inertial_params['link3']}"
-        origin_rpy="0 0 0"/>
-      <xacro:common_link_visual
-        mesh_filename="${visual_dir}/link3"
-        origin_xyz="0 0 0"
-        origin_rpy="0 0 0"
-        material_name="${prefix}White" />
-      <xacro:common_link_collision
-        mesh_filename="${collision_dir}/link3"
-        add_mesh_suffix="${add_mesh_suffix}"
-        other_mesh_suffix="${collison_mesh_suffix}"
-        origin_xyz="0 0 0"
-        origin_rpy="0 0 0" />
-    </link>
     <joint name="${prefix}joint3" type="revolute">
       <parent link="${prefix}link2"/>
@@ -167,20 +216,4 @@
       <dynamics damping="1.0" friction="1.0"/>
     </joint>
-    <link name="${prefix}link4">
-      <xacro:common_link_inertial
-        link_inertial_params="${inertial_params['link4']}"
-        origin_rpy="0 0 0"/>
-      <xacro:common_link_visual
-        mesh_filename="${visual_dir}/link4"
-        origin_xyz="0 0 0"
-        origin_rpy="0 0 0"
-        material_name="${prefix}White" />
-      <xacro:common_link_collision
-        mesh_filename="${collision_dir}/link4"
-        add_mesh_suffix="${add_mesh_suffix}"
-        other_mesh_suffix="${collison_mesh_suffix}"
-        origin_xyz="0 0 0"
-        origin_rpy="0 0 0" />
-    </link>
     <joint name="${prefix}joint4" type="revolute">
       <parent link="${prefix}link3"/>
@@ -196,20 +229,4 @@
       <dynamics damping="1.0" friction="1.0"/>
     </joint>
-    <link name="${prefix}link5">
-      <xacro:common_link_inertial
-        link_inertial_params="${inertial_params['link5']}"
-        origin_rpy="0 0 0"/>
-      <xacro:common_link_visual
-        mesh_filename="${visual_dir}/link5"
-        origin_xyz="0 0 0"
-        origin_rpy="0 0 0"
-        material_name="${prefix}White" />
-      <xacro:common_link_collision
-        mesh_filename="${collision_dir}/link5"
-        add_mesh_suffix="${add_mesh_suffix}"
-        other_mesh_suffix="${collison_mesh_suffix}"
-        origin_xyz="0 0 0"
-        origin_rpy="0 0 0" />
-    </link>
     <joint name="${prefix}joint5" type="revolute">
       <parent link="${prefix}link4"/>
@@ -224,20 +241,4 @@
       <dynamics damping="1.0" friction="1.0"/>
     </joint>
-    <link name="${prefix}link6">
-      <xacro:common_link_inertial
-        link_inertial_params="${inertial_params['link6']}"
-        origin_rpy="0 0 0"/>
-      <xacro:common_link_visual
-        mesh_filename="${link6_visual}"
-        origin_xyz="0 0 0"
-        origin_rpy="0 0 0"
-        material_name="${prefix}Silver" />
-      <xacro:common_link_collision
-        mesh_filename="${link6_collision}"
-        add_mesh_suffix="${add_mesh_suffix}"
-        other_mesh_suffix="${collison_mesh_suffix}"
-        origin_xyz="0 0 0"
-        origin_rpy="0 0 0" />
-    </link>
     <joint name="${prefix}joint6" type="revolute">
       <parent link="${prefix}link5"/>
@@ -259,4 +260,28 @@
       <child link="${prefix}link_eef" />
     </joint> -->
+    <!-- Gazebo -->
+    <xacro:if value="${use_gazebo}">
+      <gazebo reference="${prefix}base_link">
+            <selfCollide>true</selfCollide>
+        </gazebo>
+        <gazebo reference="${prefix}link1">
+            <selfCollide>true</selfCollide>
+        </gazebo>
+        <gazebo reference="${prefix}link2">
+            <selfCollide>true</selfCollide>
+        </gazebo>
+        <gazebo reference="${prefix}link3">
+            <selfCollide>true</selfCollide>
+        </gazebo>
+        <gazebo reference="${prefix}link4">
+            <selfCollide>true</selfCollide>
+        </gazebo>
+        <gazebo reference="${prefix}link5">
+            <selfCollide>true</selfCollide>
+        </gazebo>
+        <gazebo reference="${prefix}link6">
+            <selfCollide>true</selfCollide>
+        </gazebo>
+    </xacro:if>
   </xacro:macro>
 </robot>

File: husky_xarm6_mcr_description/urdf/xarm6/xarm6_ros2_control.xacro (robot description, xacro)
@@ -1,6 +1,6 @@
 <?xml version="1.0"?>
 <robot xmlns:xacro="http://ros.org/wiki/xacro">
-    <xacro:macro name="xarm6_ros2_control" params="prefix sim:=true">
-        <xacro:if value="${sim}">
+    <xacro:macro name="xarm6_ros2_control" params="prefix use_gazebo:=true">
+        <xacro:if value="${use_gazebo}">
             <ros2_control name="${prefix}gazebo_system" type="system">
                 <hardware>
@@ -46,6 +46,6 @@
             </ros2_control>
         </xacro:if>
-        <xacro:unless value="${sim}">
-            <!-- Real hardware (later) -->
+        <!-- Real hardware (later) -->
+        <!-- <xacro:unless value="${use_gazebo}">
             <ros2_control name="${prefix}uf_hw" type="system">
                 <hardware>
@@ -87,5 +87,5 @@
                 </joint>
             </ros2_control>
-        </xacro:unless>
+        </xacro:unless> -->
     </xacro:macro>
 </robot>

Commit message: Fixed current alignment of xarm on husky

File: husky_xarm6_mcr_description/urdf/husky_xarm6_mcr.urdf.xacro (robot description, xacro)
@@ -22,5 +22,5 @@
     <xacro:include filename="$(find husky_xarm6_mcr_description)/urdf/xarm6/xarm6_macro.urdf.xacro"/>
     <xacro:xarm6 namespace="$(arg manipulator_ns)" prefix="$(arg manipulator_prefix)" model_num="1303" parent_link="$(arg platform_ns)/$(arg platform_prefix)x_rail_riser_link">
-        <origin xyz="0.09500000 0 0.31610000" rpy="0 0 ${-pi/2}"/>
+        <origin xyz="0.09500000 0 0.31610000" rpy="0 0 0"/>
     </xacro:xarm6>
     <!-- ROS2_CONTROL -->
