Commit message: removed old moveit, re-implemented description package, working on the control package

File: husky_xarm6_mcr_description/srdf/husky_xarm6_mcr.srdf.xacro (robot description, xacro)
@@ -1,75 +1,92 @@
 <?xml version="1.0" encoding="UTF-8"?>
-<robot xmlns="http://www.ros.org" xmlns:xacro="http://ros.org/wiki/xacro" name="husky_xarm6_mcr">
-    <!-- invoke the xarm6 group macro -->
-    <xacro:include filename="$(find xarm_moveit_config)/srdf/_xarm6_macro.srdf.xacro"/>
-    <xacro:xarm6_macro_srdf prefix="xarm_"
-        add_gripper="false"
-        add_bio_gripper="false"
-        add_vacuum_gripper="false"
-        add_other_geometry="false"/>
+<robot xmlns:xacro="http://wiki.ros.org/xacro" name="husky_xarm6_mcr">
+    <!-- parameters -->
+    <xacro:arg name="platform_prefix" default="a200_" />
+    <xacro:arg name="manipulator_prefix" default="xarm6_" />
     <!--GROUPS: Representation of a set of joints and links. This can be useful for specifying DOF to plan for, defining arms, end effectors, etc-->
+    <group name="${platform_prefix}platform">
+        <joint name="${platform_prefix}world_joint" />
+        <joint name="${platform_prefix}front_left_wheel_joint" />
+        <joint name="${platform_prefix}front_right_wheel_joint" />
+        <joint name="${platform_prefix}rear_left_wheel_joint" />
+        <joint name="${platform_prefix}rear_right_wheel_joint" />
+    </group>
+    <group name="${manipulator_prefix}manipulator">
+        <joint name="${manipulator_prefix}joint_base_fixed" />
+        <joint name="${manipulator_prefix}joint1" />
+        <joint name="${manipulator_prefix}joint2" />
+        <joint name="${manipulator_prefix}joint3" />
+        <joint name="${manipulator_prefix}joint4" />
+        <joint name="${manipulator_prefix}joint5" />
+        <joint name="${manipulator_prefix}joint6" />
+    </group>
+    <!-- <group name="camera_rig">
+        <link name="zed2i_camera_center"/>
+        <link name="ximea_camera_link"/>
+        <link name="ffs_camera_link"/>
+        <link name="multi_camera_rig_link"/>
+    </group> -->
     <!--LINKS: When a link is specified, the parent joint of that link (if it exists) is automatically included-->
     <!--JOINTS: When a joint is specified, the child link of that joint (which will always exist) is automatically included-->
     <!--CHAINS: When a chain is specified, all the links along the chain (including endpoints) are included in the group. Additionally, all the joints that are parents to included links are also included. This means that joints along the chain and the parent joint of the base link are included in the group-->
     <!--SUBGROUPS: Groups can also be formed by referencing to already defined group names-->
-    <group name="xarm_manipulator">
-        <chain base_link="xarm_joint1" tip_link="xarm_link_eef"/>
-    </group>
-    <group name="camera_rig">
-        <link name="zed2i_camera_center"/>
-        <link name="ximea_camera_link"/>
-        <link name="ffs_camera_link"/>
-        <link name="multi_camera_rig_link"/>
-    </group>
-    <!--GROUP STATES: Purpose: Define a named state for a particular group, in terms of joint values. This is useful to define states like 'folded arms'-->
-    <group_state name="home" group="xarm_manipulator">
-        <joint name="xarm_joint1" value="0"/>
-        <joint name="xarm_joint2" value="-1.5707"/>
-        <joint name="xarm_joint3" value="0"/>
-        <joint name="xarm_joint4" value="-1.5707"/>
-        <joint name="xarm_joint5" value="0"/>
-        <joint name="xarm_joint6" value="0"/>
+    <!-- GROUP STATES, Purpose, Define a named state for a particular group, in terms of joint values. This is useful to define states like 'folded arms' -->
+    <group_state name="home" group="${manipulator_prefix}manipulator">
+        <joint name="${manipulator_prefix}joint1" value="0" />
+        <joint name="${manipulator_prefix}joint2" value="0" />
+        <joint name="${manipulator_prefix}joint3" value="0" />
+        <joint name="${manipulator_prefix}joint4" value="0" />
+        <joint name="${manipulator_prefix}joint5" value="0" />
+        <joint name="${manipulator_prefix}joint6" value="0" />
     </group_state>
     <!--END EFFECTOR: Purpose: Represent information about an end effector.-->
-    <end_effector name="camera_rig" parent_link="xarm_joint6" group="camera_rig"/>
+    <!-- <end_effector name="camera_rig" parent_link="xarm_link6" group="camera_rig"/> -->
     <!--DISABLE COLLISIONS: By default it is assumed that any link of the robot could potentially come into collision with any other link in the robot. This tag disables collision checking between a specified pair of links. -->
-    <disable_collisions link1="base_link" link2="front_left_wheel" reason="Adjacent"/>
-    <disable_collisions link1="base_link" link2="front_right_wheel" reason="Adjacent"/>
-    <disable_collisions link1="base_link" link2="rear_left_wheel" reason="Adjacent"/>
-    <disable_collisions link1="base_link" link2="rear_right_wheel" reason="Adjacent"/>
-    <disable_collisions link1="base_link" link2="x-rail_platform_link" reason="Adjacent"/>
-    <disable_collisions link1="ffs_camera_link" link2="ximea_camera_link" reason="Default"/>
-    <disable_collisions link1="ffs_camera_link" link2="zed2i_camera_center" reason="Never"/>
-    <disable_collisions link1="front_left_wheel" link2="front_left_wheel" reason="Default"/>
-    <disable_collisions link1="front_left_wheel" link2="front_right_wheel" reason="Never"/>
-    <disable_collisions link1="front_left_wheel" link2="rear_left_wheel" reason="Never"/>
-    <disable_collisions link1="front_left_wheel" link2="rear_right_wheel" reason="Never"/>
-    <disable_collisions link1="front_left_wheel" link2="xarm_joint1" reason="Never"/>
-    <disable_collisions link1="front_left_wheel" link2="xarm_joint2" reason="Never"/>
-    <disable_collisions link1="front_left_wheel" link2="xarm_joint3" reason="Never"/>
-    <disable_collisions link1="front_left_wheel" link2="x-rail_platform_link" reason="Never"/>
-    <disable_collisions link1="front_right_wheel" link2="front_right_wheel" reason="Default"/>
-    <disable_collisions link1="front_right_wheel" link2="rear_left_wheel" reason="Never"/>
-    <disable_collisions link1="front_right_wheel" link2="rear_right_wheel" reason="Never"/>
-    <disable_collisions link1="front_right_wheel" link2="xarm_joint1" reason="Never"/>
-    <disable_collisions link1="front_right_wheel" link2="xarm_joint2" reason="Never"/>
-    <disable_collisions link1="front_right_wheel" link2="xarm_joint3" reason="Never"/>
-    <disable_collisions link1="front_right_wheel" link2="x-rail_platform_link" reason="Never"/>
-    <disable_collisions link1="multi_camera_rig_link" link2="xarm_joint4" reason="Never"/>
-    <disable_collisions link1="multi_camera_rig_link" link2="xarm_joint5" reason="Never"/>
-    <disable_collisions link1="multi_camera_rig_link" link2="xarm_joint6" reason="Adjacent"/>
-    <disable_collisions link1="multi_camera_rig_link" link2="ximea_camera_link" reason="Adjacent"/>
-    <disable_collisions link1="multi_camera_rig_link" link2="zed2i_camera_center" reason="Adjacent"/>
-    <disable_collisions link1="multi_camera_rig_link" link2="ffs_camera_link" reason="Adjacent"/>
-    <disable_collisions link1="rear_left_wheel" link2="rear_left_wheel" reason="Default"/>
-    <disable_collisions link1="rear_left_wheel" link2="rear_right_wheel" reason="Never"/>
-    <disable_collisions link1="rear_left_wheel" link2="xarm_joint1" reason="Never"/>
-    <disable_collisions link1="rear_left_wheel" link2="xarm_joint2" reason="Never"/>
-    <disable_collisions link1="rear_left_wheel" link2="xarm_joint3" reason="Never"/>
-    <disable_collisions link1="rear_left_wheel" link2="x-rail_platform_link" reason="Never"/>
-    <disable_collisions link1="rear_right_wheel" link2="rear_right_wheel" reason="Default"/>
-    <disable_collisions link1="rear_right_wheel" link2="xarm_joint1" reason="Never"/>
-    <disable_collisions link1="rear_right_wheel" link2="xarm_joint2" reason="Never"/>
-    <disable_collisions link1="rear_right_wheel" link2="xarm_joint3" reason="Never"/>
-    <disable_collisions link1="rear_right_wheel" link2="x-rail_platform_link" reason="Never"/>
+    <!-- Platform collisions -->
+    <disable_collisions link1="${platform_prefix}base_link" link2="${platform_prefix}front_left_wheel" reason="Adjacent"/>
+    <disable_collisions link1="${platform_prefix}base_link" link2="${platform_prefix}front_right_wheel" reason="Adjacent"/>
+    <disable_collisions link1="${platform_prefix}base_link" link2="${platform_prefix}rear_left_wheel" reason="Adjacent"/>
+    <disable_collisions link1="${platform_prefix}base_link" link2="${platform_prefix}rear_right_wheel" reason="Adjacent"/>
+    <disable_collisions link1="${platform_prefix}base_link" link2="x_rail_riser_link" reason="Adjacent"/>
+    <!-- Manipulator base link collisions -->
+    <disable_collisions link1="${manipulator_prefix}base_link" link2="${platform_prefix}front_left_wheel" reason="Never"/>
+    <disable_collisions link1="${manipulator_prefix}base_link" link2="${platform_prefix}front_right_wheel" reason="Never"/>
+    <disable_collisions link1="${manipulator_prefix}base_link" link2="${platform_prefix}rear_left_wheel" reason="Never"/>
+    <disable_collisions link1="${manipulator_prefix}base_link" link2="${platform_prefix}rear_right_wheel" reason="Never"/>
+    <disable_collisions link1="${manipulator_prefix}base_link" link2="${platform_prefix}base_link" reason="Never"/>
+    <disable_collisions link1="${manipulator_prefix}base_link" link2="x_rail_riser_link" reason="adjacent"/>
+    <disable_collisions link1="${manipulator_prefix}base_link" link2="${manipulator_prefix}link1" reason="adjacent"/>
+    <disable_collisions link1="${manipulator_prefix}base_link" link2="${manipulator_prefix}link2" reason="Never"/>
+    <!-- Manipulator link1 collisions -->
+    <disable_collisions link1="${manipulator_prefix}link1" link2="${platform_prefix}front_left_wheel" reason="Never"/>
+    <disable_collisions link1="${manipulator_prefix}link1" link2="${platform_prefix}front_right_wheel" reason="Never"/>
+    <disable_collisions link1="${manipulator_prefix}link1" link2="${platform_prefix}rear_left_wheel" reason="Never"/>
+    <disable_collisions link1="${manipulator_prefix}link1" link2="${platform_prefix}rear_right_wheel" reason="Never"/>
+    <disable_collisions link1="${manipulator_prefix}link1" link2="${platform_prefix}base_link" reason="Never"/>
+    <disable_collisions link1="${manipulator_prefix}link1" link2="x_rail_riser_link" reason="Never"/>
+    <disable_collisions link1="${manipulator_prefix}link1" link2="${manipulator_prefix}link2" reason="adjacent"/>
+    <disable_collisions link1="${manipulator_prefix}link1" link2="${manipulator_prefix}link3" reason="Never"/>
+    <!-- Manipulator link2 collisions -->
+    <disable_collisions link1="${manipulator_prefix}link2" link2="${platform_prefix}front_left_wheel" reason="Never"/>
+    <disable_collisions link1="${manipulator_prefix}link2" link2="${platform_prefix}front_right_wheel" reason="Never"/>
+    <disable_collisions link1="${manipulator_prefix}link2" link2="${platform_prefix}rear_left_wheel" reason="Never"/>
+    <disable_collisions link1="${manipulator_prefix}link2" link2="${platform_prefix}rear_right_wheel" reason="Never"/>
+    <disable_collisions link1="${manipulator_prefix}link2" link2="${platform_prefix}base_link" reason="Never"/>
+    <disable_collisions link1="${manipulator_prefix}link2" link2="x_rail_riser_link" reason="Never"/>
+    <disable_collisions link1="${manipulator_prefix}link2" link2="${manipulator_prefix}link3" reason="adjacent"/>
+    <disable_collisions link1="${manipulator_prefix}link2" link2="${manipulator_prefix}link4" reason="Never"/>
+    <!-- Manipulator link3 collisions -->
+    <disable_collisions link1="${manipulator_prefix}link3" link2="${platform_prefix}front_left_wheel" reason="Never"/>
+    <disable_collisions link1="${manipulator_prefix}link3" link2="${platform_prefix}front_right_wheel" reason="Never"/>
+    <disable_collisions link1="${manipulator_prefix}link3" link2="${platform_prefix}rear_left_wheel" reason="Never"/>
+    <disable_collisions link1="${manipulator_prefix}link3" link2="${platform_prefix}rear_right_wheel" reason="Never"/>
+    <disable_collisions link1="${manipulator_prefix}link3" link2="${platform_prefix}base_link" reason="Never"/>
+    <disable_collisions link1="${manipulator_prefix}link3" link2="${manipulator_prefix}link4" reason="adjacent"/>
+    <disable_collisions link1="${manipulator_prefix}link3" link2="${manipulator_prefix}link5" reason="Never"/>
+    <!-- Manipulator link4 collisions -->
+    <disable_collisions link1="${manipulator_prefix}link4" link2="${manipulator_prefix}link5" reason="adjacent"/>
+    <disable_collisions link1="${manipulator_prefix}link4" link2="${manipulator_prefix}link6" reason="Never"/>
+    <!-- Manipulator link5 collisions -->
+    <disable_collisions link1="${manipulator_prefix}link5" link2="${manipulator_prefix}link6" reason="adjacent"/>
+    <!-- Manipulator link6 collisions -->
 </robot>

File: husky_xarm6_mcr_description/urdf/husky_xarm6_mcr.urdf.xacro (robot description, xacro)
@@ -1,74 +1,38 @@
-<?xml version="1.0"?>
+<?xml version='1.0' encoding='utf-8'?>
 <robot xmlns:xacro="http://ros.org/wiki/xacro" name="husky_xarm6_mcr">
+    <!-- Arguments -->
+    <xacro:arg name="sim" default="true"/>
+    <xacro:arg name="manipulator_prefix" default="xarm6_"/>
+    <xacro:arg name="platform_prefix" default="a200_"/>
     <!-- Parameters -->
     <!-- HUSKY PLATFORM & ATTACHMENTS -->
-    <!-- Husky body -->
-    <xacro:include filename="$(find clearpath_platform_description)/urdf/common.urdf.xacro"/>
-    <xacro:include filename="$(find clearpath_platform_description)/urdf/a200/a200.urdf.xacro"/>
-    <xacro:a200 wheel="default"/>
-    <!-- front & rear bumper -->
-    <xacro:include filename="$(find clearpath_platform_description)/urdf/a200/attachments/bumper.urdf.xacro"/>
-    <xacro:bumper name="front_bumper"
-                model="default"
-                parent_link="front_bumper_mount">
-        <origin xyz="0 0 0" rpy="0 0 0"/>
-    </xacro:bumper>
-    <xacro:bumper name="rear_bumper"
-                model="default"
-                parent_link="rear_bumper_mount">
-        <origin xyz="0 0 0" rpy="0 0 0"/>
-    </xacro:bumper>
-    <!-- X-RAIL PLATFORM -->
-    <link name="x-rail_platform_link">
-        <visual>
-            <origin xyz="0 0 0" rpy="0 0 0"/>
-            <geometry>
-                <mesh filename="package://husky_xarm6_mcr_description/meshes/Platform_Electronics.dae" scale="1 1 1"/>
-            </geometry>
-        </visual>
-        <collision>
-            <origin xyz="0 0 0" rpy="0 0 0"/>
-            <geometry>
-                <mesh filename="package://husky_xarm6_mcr_description/meshes/Platform_Electronics_Collision.stl" scale="1 1 1"/>
-            </geometry>
-        </collision>
-        <!-- <inertial>
-            <origin xyz="0.01142856 0.38887557 0.14875439" rpy="0 0 0"/>
-            <mass value="37.70490883"/>
-            <inertia
-                ixx="3.0863383" ixy="0.13633027" ixz="-0.05595213"
-                iyy="1.23426261" iyz="0.14585405"
-                izz="3.73292102"/>
-        </inertial> -->
-    </link>
-    <joint name="x-rail_husky_joint" type="fixed">
-        <parent link="base_link"/>
-        <child link="x-rail_platform_link"/>
-        <origin xyz="0.0 0.0 0.24020000" rpy="0 0 ${-pi/2}"/>
-    </joint>
+    <xacro:include filename="$(find husky_xarm6_mcr_description)/urdf/husky/a200_macro.urdf.xacro"/>
+    <xacro:a200 prefix="$(arg platform_prefix)"/>
+    <!-- X-RAIL RISER -->
+    <xacro:include filename="$(find husky_xarm6_mcr_description)/urdf/risers/x_rail_macro.urdf.xacro"/>
+    <xacro:x_rail_riser prefix="" parent_link="a200_default_mount">
+        <origin xyz="0.0 0.0 0.0" rpy="0 0 ${-pi/2}"/>
+    </xacro:x_rail_riser>
+    <!-- ROS2_CONTROL -->
+    <xacro:include filename="$(find husky_xarm6_mcr_description)/urdf/husky/husky_ros2_control.xacro"/>
+    <xacro:husky_ros2_control
+        use_gazebo="$(arg sim)"
+        front_left_wheel_joint="$(arg platform_prefix)front_left_wheel_joint"
+        rear_left_wheel_joint="$(arg platform_prefix)rear_left_wheel_joint"
+        front_right_wheel_joint="$(arg platform_prefix)front_right_wheel_joint"
+        rear_right_wheel_joint="$(arg platform_prefix)rear_right_wheel_joint"
+    />
+    <gazebo>
+        <plugin filename="gz_ros2_control-system" name="gz_ros2_control::GazeboSimROS2ControlPlugin">
+            <parameters>$(find husky_xarm6_mcr_control)/config/controllers.yaml</parameters>
+        </plugin>
+    </gazebo>
     <!-- XARM6 -->
-    <xacro:include filename="$(find xarm_description)/urdf/xarm_device_macro.xacro"/>
-    <xacro:xarm_device
-        prefix="xarm_"
-        hw_ns="xarm"
-        dof="6"
-        robot_type="xarm"
-        attach_to="x-rail_platform_link"
-        attach_xyz="0.09500000 0 0.31610000"
-        attach_rpy="0 0 ${-pi/2}"
-        create_attach_link="false"
-        limited="false"
-        effort_control="false"
-        velocity_control="false"
-        ros2_control_plugin="uf_robot_hardware/UFRobotSystemHardware"
-        ros2_control_params=""
-        load_gazebo_plugin="false"
-        add_gripper="false"
-        add_vacuum_gripper="false"
-        add_bio_gripper="false"
-        model1300="false"
-    />
+    <!-- <xacro:include filename="$(find husky_xarm6_mcr_description)/urdf/xarm6/xarm6_macro.urdf.xacro"/>
+    <xacro:xarm6 prefix="$(arg manipulator_prefix)" model_num="1303" parent_link="x_rail_riser_link">
+        <origin xyz="0.09500000 0 0.31610000" rpy="0 0 ${-pi/2}"/>
+    </xacro:xarm6> -->
     <!-- MULTI CAMERA RIG -->
-    <xacro:include filename="$(find multi_cam_rig_description)/urdf/multi_cam_rig_macro.urdf.xacro"/>
+    <!-- <xacro:include filename="$(find multi_cam_rig_description)/urdf/multi_cam_rig_macro.urdf.xacro"/>
     <xacro:multi_camera_rig/>
     <joint name="tool_mount" type="fixed">
@@ -76,4 +40,18 @@
         <child link="multi_camera_rig_link"/>
         <origin xyz="0.0 0.0 0.0" rpy="${pi/2} 0 0"/>
-    </joint>
+    </joint> -->
+    <!-- ROS2_CONTROL -->
+    <!-- HUSKY ros2_control block (binds joints(arg to hardware) -->
+    <!-- <xacro:include filename="$(find husky_xarm6_mcr_description)/urdf/xarm6/xarm6_ros2_control.xacro"/>
+    <xacro:xarm6_ros2_control prefix="$(arg manipulator_prefix)" sim="$(arg sim)"/>
+    <gazebo>
+        <plugin filename="gz_ros2_control-system" name="gz_ros2_control::GazeboSimROS2ControlPlugin">
+            <robot_param>robot_description</robot_param>
+            <robot_param_node>robot_state_publisher</robot_param_node>
+            <parameters>$(find husky_xarm6_mcr_control)/config/controllers.yaml</parameters>
+        </plugin>
+    </gazebo> -->
+    <!-- Gazebo -->
+    <!-- <xacro:include filename="$(find husky_xarm6_mcr_description)/urdf/xarm6/xarm6_gazebo.xacro"/>
+    <xacro:xarm6_gazebo prefix="$(arg manipulator_prefix)"/> -->
 </robot>
