Commit message: Add bringup package, apple orchard simulation env, and moveit config with Git LFS for large mesh files

File: husky_xarm6_mcr_description/srdf/husky_xarm6_mcr.srdf.xacro (robot description, xacro)
@@ -1,23 +1,22 @@
-<?xml version="1.0" encoding="UTF-8"?>
-<robot xmlns:xacro="http://wiki.ros.org/xacro" name="husky_xarm6_mcr">
+<?xml version='1.0' encoding='utf-8'?>
+<robot xmlns:xacro="http://ros.org/wiki/xacro" name="husky_xarm6_mcr">
     <!-- parameters -->
-    <xacro:arg name="platform_prefix" default="a200_" />
-    <xacro:arg name="manipulator_prefix" default="xarm6_" />
+    <xacro:arg name="manipulator_prefix" default="xarm6_"/>
+    <xacro:arg name="platform_prefix" default="a200_"/>
     <!--GROUPS: Representation of a set of joints and links. This can be useful for specifying DOF to plan for, defining arms, end effectors, etc-->
-    <group name="${platform_prefix}platform">
-        <joint name="${platform_prefix}world_joint" />
-        <joint name="${platform_prefix}front_left_wheel_joint" />
-        <joint name="${platform_prefix}front_right_wheel_joint" />
-        <joint name="${platform_prefix}rear_left_wheel_joint" />
-        <joint name="${platform_prefix}rear_right_wheel_joint" />
+    <group name="$(arg platform_prefix)platform">
+        <joint name="$(arg platform_prefix)front_left_wheel_joint" />
+        <joint name="$(arg platform_prefix)front_right_wheel_joint" />
+        <joint name="$(arg platform_prefix)rear_left_wheel_joint" />
+        <joint name="$(arg platform_prefix)rear_right_wheel_joint" />
     </group>
-    <group name="${manipulator_prefix}manipulator">
-        <joint name="${manipulator_prefix}joint_base_fixed" />
-        <joint name="${manipulator_prefix}joint1" />
-        <joint name="${manipulator_prefix}joint2" />
-        <joint name="${manipulator_prefix}joint3" />
-        <joint name="${manipulator_prefix}joint4" />
-        <joint name="${manipulator_prefix}joint5" />
-        <joint name="${manipulator_prefix}joint6" />
+    <group name="$(arg manipulator_prefix)manipulator"> <!--Has to match in the kinematics and ompl_planning config files-->
+        <joint name="$(arg manipulator_prefix)joint_base_fixed" />
+        <joint name="$(arg manipulator_prefix)joint1" />
+        <joint name="$(arg manipulator_prefix)joint2" />
+        <joint name="$(arg manipulator_prefix)joint3" />
+        <joint name="$(arg manipulator_prefix)joint4" />
+        <joint name="$(arg manipulator_prefix)joint5" />
+        <joint name="$(arg manipulator_prefix)joint6" />
     </group>
     <!-- <group name="camera_rig">
@@ -32,11 +31,11 @@
     <!--SUBGROUPS: Groups can also be formed by referencing to already defined group names-->
     <!-- GROUP STATES, Purpose, Define a named state for a particular group, in terms of joint values. This is useful to define states like 'folded arms' -->
-    <group_state name="home" group="${manipulator_prefix}manipulator">
-        <joint name="${manipulator_prefix}joint1" value="0" />
-        <joint name="${manipulator_prefix}joint2" value="0" />
-        <joint name="${manipulator_prefix}joint3" value="0" />
-        <joint name="${manipulator_prefix}joint4" value="0" />
-        <joint name="${manipulator_prefix}joint5" value="0" />
-        <joint name="${manipulator_prefix}joint6" value="0" />
+    <group_state name="home" group="$(arg manipulator_prefix)manipulator">
+        <joint name="$(arg manipulator_prefix)joint1" value="0" />
+        <joint name="$(arg manipulator_prefix)joint2" value="0" />
+        <joint name="$(arg manipulator_prefix)joint3" value="0" />
+        <joint name="$(arg manipulator_prefix)joint4" value="0" />
+        <joint name="$(arg manipulator_prefix)joint5" value="0" />
+        <joint name="$(arg manipulator_prefix)joint6" value="0" />
     </group_state>
     <!--END EFFECTOR: Purpose: Represent information about an end effector.-->
@@ -44,49 +43,49 @@
     <!--DISABLE COLLISIONS: By default it is assumed that any link of the robot could potentially come into collision with any other link in the robot. This tag disables collision checking between a specified pair of links. -->
     <!-- Platform collisions -->
-    <disable_collisions link1="${platform_prefix}base_link" link2="${platform_prefix}front_left_wheel" reason="Adjacent"/>
-    <disable_collisions link1="${platform_prefix}base_link" link2="${platform_prefix}front_right_wheel" reason="Adjacent"/>
-    <disable_collisions link1="${platform_prefix}base_link" link2="${platform_prefix}rear_left_wheel" reason="Adjacent"/>
-    <disable_collisions link1="${platform_prefix}base_link" link2="${platform_prefix}rear_right_wheel" reason="Adjacent"/>
-    <disable_collisions link1="${platform_prefix}base_link" link2="x_rail_riser_link" reason="Adjacent"/>
+    <disable_collisions link1="$(arg platform_prefix)base_link" link2="$(arg platform_prefix)front_left_wheel" reason="Adjacent"/>
+    <disable_collisions link1="$(arg platform_prefix)base_link" link2="$(arg platform_prefix)front_right_wheel" reason="Adjacent"/>
+    <disable_collisions link1="$(arg platform_prefix)base_link" link2="$(arg platform_prefix)rear_left_wheel" reason="Adjacent"/>
+    <disable_collisions link1="$(arg platform_prefix)base_link" link2="$(arg platform_prefix)rear_right_wheel" reason="Adjacent"/>
+    <disable_collisions link1="$(arg platform_prefix)base_link" link2="x_rail_riser_link" reason="Adjacent"/>
     <!-- Manipulator base link collisions -->
-    <disable_collisions link1="${manipulator_prefix}base_link" link2="${platform_prefix}front_left_wheel" reason="Never"/>
-    <disable_collisions link1="${manipulator_prefix}base_link" link2="${platform_prefix}front_right_wheel" reason="Never"/>
-    <disable_collisions link1="${manipulator_prefix}base_link" link2="${platform_prefix}rear_left_wheel" reason="Never"/>
-    <disable_collisions link1="${manipulator_prefix}base_link" link2="${platform_prefix}rear_right_wheel" reason="Never"/>
-    <disable_collisions link1="${manipulator_prefix}base_link" link2="${platform_prefix}base_link" reason="Never"/>
-    <disable_collisions link1="${manipulator_prefix}base_link" link2="x_rail_riser_link" reason="adjacent"/>
-    <disable_collisions link1="${manipulator_prefix}base_link" link2="${manipulator_prefix}link1" reason="adjacent"/>
-    <disable_collisions link1="${manipulator_prefix}base_link" link2="${manipulator_prefix}link2" reason="Never"/>
+    <disable_collisions link1="$(arg manipulator_prefix)base_link" link2="$(arg platform_prefix)front_left_wheel" reason="Never"/>
+    <disable_collisions link1="$(arg manipulator_prefix)base_link" link2="$(arg platform_prefix)front_right_wheel" reason="Never"/>
+    <disable_collisions link1="$(arg manipulator_prefix)base_link" link2="$(arg platform_prefix)rear_left_wheel" reason="Never"/>
+    <disable_collisions link1="$(arg manipulator_prefix)base_link" link2="$(arg platform_prefix)rear_right_wheel" reason="Never"/>
+    <disable_collisions link1="$(arg manipulator_prefix)base_link" link2="$(arg platform_prefix)base_link" reason="Never"/>
+    <disable_collisions link1="$(arg manipulator_prefix)base_link" link2="x_rail_riser_link" reason="adjacent"/>
+    <disable_collisions link1="$(arg manipulator_prefix)base_link" link2="$(arg manipulator_prefix)link1" reason="adjacent"/>
+    <disable_collisions link1="$(arg manipulator_prefix)base_link" link2="$(arg manipulator_prefix)link2" reason="Never"/>
     <!-- Manipulator link1 collisions -->
-    <disable_collisions link1="${manipulator_prefix}link1" link2="${platform_prefix}front_left_wheel" reason="Never"/>
-    <disable_collisions link1="${manipulator_prefix}link1" link2="${platform_prefix}front_right_wheel" reason="Never"/>
-    <disable_collisions link1="${manipulator_prefix}link1" link2="${platform_prefix}rear_left_wheel" reason="Never"/>
-    <disable_collisions link1="${manipulator_prefix}link1" link2="${platform_prefix}rear_right_wheel" reason="Never"/>
-    <disable_collisions link1="${manipulator_prefix}link1" link2="${platform_prefix}base_link" reason="Never"/>
-    <disable_collisions link1="${manipulator_prefix}link1" link2="x_rail_riser_link" reason="Never"/>
-    <disable_collisions link1="${manipulator_prefix}link1" link2="${manipulator_prefix}link2" reason="adjacent"/>
-    <disable_collisions link1="${manipulator_prefix}link1" link2="${manipulator_prefix}link3" reason="Never"/>
+    <disable_collisions link1="$(arg manipulator_prefix)link1" link2="$(arg platform_prefix)front_left_wheel" reason="Never"/>
+    <disable_collisions link1="$(arg manipulator_prefix)link1" link2="$(arg platform_prefix)front_right_wheel" reason="Never"/>
+    <disable_collisions link1="$(arg manipulator_prefix)link1" link2="$(arg platform_prefix)rear_left_wheel" reason="Never"/>
+    <disable_collisions link1="$(arg manipulator_prefix)link1" link2="$(arg platform_prefix)rear_right_wheel" reason="Never"/>
+    <disable_collisions link1="$(arg manipulator_prefix)link1" link2="$(arg platform_prefix)base_link" reason="Never"/>
+    <disable_collisions link1="$(arg manipulator_prefix)link1" link2="x_rail_riser_link" reason="Never"/>
+    <disable_collisions link1="$(arg manipulator_prefix)link1" link2="$(arg manipulator_prefix)link2" reason="adjacent"/>
+    <disable_collisions link1="$(arg manipulator_prefix)link1" link2="$(arg manipulator_prefix)link3" reason="Never"/>
     <!-- Manipulator link2 collisions -->
-    <disable_collisions link1="${manipulator_prefix}link2" link2="${platform_prefix}front_left_wheel" reason="Never"/>
-    <disable_collisions link1="${manipulator_prefix}link2" link2="${platform_prefix}front_right_wheel" reason="Never"/>
-    <disable_collisions link1="${manipulator_prefix}link2" link2="${platform_prefix}rear_left_wheel" reason="Never"/>
-    <disable_collisions link1="${manipulator_prefix}link2" link2="${platform_prefix}rear_right_wheel" reason="Never"/>
-    <disable_collisions link1="${manipulator_prefix}link2" link2="${platform_prefix}base_link" reason="Never"/>
-    <disable_collisions link1="${manipulator_prefix}link2" link2="x_rail_riser_link" reason="Never"/>
-    <disable_collisions link1="${manipulator_prefix}link2" link2="${manipulator_prefix}link3" reason="adjacent"/>
-    <disable_collisions link1="${manipulator_prefix}link2" link2="${manipulator_prefix}link4" reason="Never"/>
+    <disable_collisions link1="$(arg manipulator_prefix)link2" link2="$(arg platform_prefix)front_left_wheel" reason="Never"/>
+    <disable_collisions link1="$(arg manipulator_prefix)link2" link2="$(arg platform_prefix)front_right_wheel" reason="Never"/>
+    <disable_collisions link1="$(arg manipulator_prefix)link2" link2="$(arg platform_prefix)rear_left_wheel" reason="Never"/>
+    <disable_collisions link1="$(arg manipulator_prefix)link2" link2="$(arg platform_prefix)rear_right_wheel" reason="Never"/>
+    <disable_collisions link1="$(arg manipulator_prefix)link2" link2="$(arg platform_prefix)base_link" reason="Never"/>
+    <disable_collisions link1="$(arg manipulator_prefix)link2" link2="x_rail_riser_link" reason="Never"/>
+    <disable_collisions link1="$(arg manipulator_prefix)link2" link2="$(arg manipulator_prefix)link3" reason="adjacent"/>
+    <disable_collisions link1="$(arg manipulator_prefix)link2" link2="$(arg manipulator_prefix)link4" reason="Never"/>
     <!-- Manipulator link3 collisions -->
-    <disable_collisions link1="${manipulator_prefix}link3" link2="${platform_prefix}front_left_wheel" reason="Never"/>
-    <disable_collisions link1="${manipulator_prefix}link3" link2="${platform_prefix}front_right_wheel" reason="Never"/>
-    <disable_collisions link1="${manipulator_prefix}link3" link2="${platform_prefix}rear_left_wheel" reason="Never"/>
-    <disable_collisions link1="${manipulator_prefix}link3" link2="${platform_prefix}rear_right_wheel" reason="Never"/>
-    <disable_collisions link1="${manipulator_prefix}link3" link2="${platform_prefix}base_link" reason="Never"/>
-    <disable_collisions link1="${manipulator_prefix}link3" link2="${manipulator_prefix}link4" reason="adjacent"/>
-    <disable_collisions link1="${manipulator_prefix}link3" link2="${manipulator_prefix}link5" reason="Never"/>
+    <disable_collisions link1="$(arg manipulator_prefix)link3" link2="$(arg platform_prefix)front_left_wheel" reason="Never"/>
+    <disable_collisions link1="$(arg manipulator_prefix)link3" link2="$(arg platform_prefix)front_right_wheel" reason="Never"/>
+    <disable_collisions link1="$(arg manipulator_prefix)link3" link2="$(arg platform_prefix)rear_left_wheel" reason="Never"/>
+    <disable_collisions link1="$(arg manipulator_prefix)link3" link2="$(arg platform_prefix)rear_right_wheel" reason="Never"/>
+    <disable_collisions link1="$(arg manipulator_prefix)link3" link2="$(arg platform_prefix)base_link" reason="Never"/>
+    <disable_collisions link1="$(arg manipulator_prefix)link3" link2="$(arg manipulator_prefix)link4" reason="adjacent"/>
+    <disable_collisions link1="$(arg manipulator_prefix)link3" link2="$(arg manipulator_prefix)link5" reason="Never"/>
     <!-- Manipulator link4 collisions -->
-    <disable_collisions link1="${manipulator_prefix}link4" link2="${manipulator_prefix}link5" reason="adjacent"/>
-    <disable_collisions link1="${manipulator_prefix}link4" link2="${manipulator_prefix}link6" reason="Never"/>
+    <disable_collisions link1="$(arg manipulator_prefix)link4" link2="$(arg manipulator_prefix)link5" reason="adjacent"/>
+    <disable_collisions link1="$(arg manipulator_prefix)link4" link2="$(arg manipulator_prefix)link6" reason="Never"/>
     <!-- Manipulator link5 collisions -->
-    <disable_collisions link1="${manipulator_prefix}link5" link2="${manipulator_prefix}link6" reason="adjacent"/>
+    <disable_collisions link1="$(arg manipulator_prefix)link5" link2="$(arg manipulator_prefix)link6" reason="adjacent"/>
     <!-- Manipulator link6 collisions -->
 </robot>
