Commit message: Added multi camera rig to simulation. Added initial joint positions to avoid collision at the start. Working on getting the images to show from the stereo camera in gazebo ign.

File: husky_xarm6_mcr_description/srdf/husky_xarm6_mcr.srdf.xacro (robot description, xacro)
@@ -4,4 +4,6 @@
     <xacro:arg name="manipulator_prefix" default="xarm6_"/>
     <xacro:arg name="platform_prefix" default="a200_"/>
+    <!-- Import multi camera rig SRDF -->
+    <xacro:include filename="$(find multi_cam_rig_description)/srdf/multi_cam_rig.srdf.xacro"/>
     <!--GROUPS: Representation of a set of joints and links. This can be useful for specifying DOF to plan for, defining arms, end effectors, etc-->
     <group name="$(arg platform_prefix)platform">
@@ -20,10 +22,10 @@
         <joint name="$(arg manipulator_prefix)joint6" />
     </group>
-    <!-- <group name="camera_rig">
+    <group name="camera_rig">
         <link name="zed2i_camera_center"/>
         <link name="ximea_camera_link"/>
         <link name="ffs_camera_link"/>
         <link name="multi_camera_rig_link"/>
-    </group> -->
+    </group>
     <!--LINKS: When a link is specified, the parent joint of that link (if it exists) is automatically included-->
     <!--JOINTS: When a joint is specified, the child link of that joint (which will always exist) is automatically included-->
@@ -54,6 +56,6 @@
     <disable_collisions link1="$(arg manipulator_prefix)base_link" link2="$(arg platform_prefix)rear_right_wheel" reason="Never"/>
     <disable_collisions link1="$(arg manipulator_prefix)base_link" link2="$(arg platform_prefix)base_link" reason="Never"/>
-    <disable_collisions link1="$(arg manipulator_prefix)base_link" link2="x_rail_riser_link" reason="adjacent"/>
-    <disable_collisions link1="$(arg manipulator_prefix)base_link" link2="$(arg manipulator_prefix)link1" reason="adjacent"/>
+    <disable_collisions link1="$(arg manipulator_prefix)base_link" link2="x_rail_riser_link" reason="Adjacent"/>
+    <disable_collisions link1="$(arg manipulator_prefix)base_link" link2="$(arg manipulator_prefix)link1" reason="Adjacent"/>
     <disable_collisions link1="$(arg manipulator_prefix)base_link" link2="$(arg manipulator_prefix)link2" reason="Never"/>
     <!-- Manipulator link1 collisions -->
@@ -64,5 +66,5 @@
     <disable_collisions link1="$(arg manipulator_prefix)link1" link2="$(arg platform_prefix)base_link" reason="Never"/>
     <disable_collisions link1="$(arg manipulator_prefix)link1" link2="x_rail_riser_link" reason="Never"/>
-    <disable_collisions link1="$(arg manipulator_prefix)link1" link2="$(arg manipulator_prefix)link2" reason="adjacent"/>
+    <disable_collisions link1="$(arg manipulator_prefix)link1" link2="$(arg manipulator_prefix)link2" reason="Adjacent"/>
     <disable_collisions link1="$(arg manipulator_prefix)link1" link2="$(arg manipulator_prefix)link3" reason="Never"/>
     <!-- Manipulator link2 collisions -->
@@ -73,5 +75,5 @@
     <disable_collisions link1="$(arg manipulator_prefix)link2" link2="$(arg platform_prefix)base_link" reason="Never"/>
     <disable_collisions link1="$(arg manipulator_prefix)link2" link2="x_rail_riser_link" reason="Never"/>
-    <disable_collisions link1="$(arg manipulator_prefix)link2" link2="$(arg manipulator_prefix)link3" reason="adjacent"/>
+    <disable_collisions link1="$(arg manipulator_prefix)link2" link2="$(arg manipulator_prefix)link3" reason="Adjacent"/>
     <disable_collisions link1="$(arg manipulator_prefix)link2" link2="$(arg manipulator_prefix)link4" reason="Never"/>
     <!-- Manipulator link3 collisions -->
@@ -81,11 +83,14 @@
     <disable_collisions link1="$(arg manipulator_prefix)link3" link2="$(arg platform_prefix)rear_right_wheel" reason="Never"/>
     <disable_collisions link1="$(arg manipulator_prefix)link3" link2="$(arg platform_prefix)base_link" reason="Never"/>
-    <disable_collisions link1="$(arg manipulator_prefix)link3" link2="$(arg manipulator_prefix)link4" reason="adjacent"/>
+    <disable_collisions link1="$(arg manipulator_prefix)link3" link2="$(arg manipulator_prefix)link4" reason="Adjacent"/>
     <disable_collisions link1="$(arg manipulator_prefix)link3" link2="$(arg manipulator_prefix)link5" reason="Never"/>
     <!-- Manipulator link4 collisions -->
-    <disable_collisions link1="$(arg manipulator_prefix)link4" link2="$(arg manipulator_prefix)link5" reason="adjacent"/>
+    <disable_collisions link1="$(arg manipulator_prefix)link4" link2="$(arg manipulator_prefix)link5" reason="Adjacent"/>
     <disable_collisions link1="$(arg manipulator_prefix)link4" link2="$(arg manipulator_prefix)link6" reason="Never"/>
     <!-- Manipulator link5 collisions -->
-    <disable_collisions link1="$(arg manipulator_prefix)link5" link2="$(arg manipulator_prefix)link6" reason="adjacent"/>
+    <disable_collisions link1="$(arg manipulator_prefix)link5" link2="$(arg manipulator_prefix)link6" reason="Adjacent"/>
     <!-- Manipulator link6 collisions -->
+    <disable_collisions link1="$(arg manipulator_prefix)link6" link2="multi_camera_rig_link" reason="Adjacent"/>
+    <!-- Multi camera rig collision settings -->
+    <xacro:multi_camera_rig/>
 </robot>

File: husky_xarm6_mcr_description/urdf/husky_xarm6_mcr.urdf.xacro (robot description, xacro)
@@ -10,5 +10,5 @@
     <!-- X-RAIL RISER -->
     <xacro:include filename="$(find husky_xarm6_mcr_description)/urdf/risers/x_rail_macro.urdf.xacro"/>
-    <xacro:x_rail_riser prefix="" parent_link="a200_default_mount">
+    <xacro:x_rail_riser prefix="" parent_link="$(arg platform_prefix)default_mount">
         <origin xyz="0.0 0.0 0.0" rpy="0 0 ${-pi/2}"/>
     </xacro:x_rail_riser>
@@ -29,24 +29,10 @@
     </gazebo>
     <!-- MULTI CAMERA RIG -->
-    <!-- <xacro:include filename="$(find multi_cam_rig_description)/urdf/multi_cam_rig_macro.urdf.xacro"/>
-    <xacro:multi_camera_rig/>
+    <xacro:include filename="$(find multi_cam_rig_description)/urdf/multi_cam_rig_macro.urdf.xacro"/>
+    <xacro:multi_camera_rig use_gazebo="$(arg sim)"/>
     <joint name="tool_mount" type="fixed">
-        <parent link="xarm_link_eef"/>
-        <child link="multi_camera_rig_link"/>
+        <parent link="$(arg manipulator_prefix)link_eef"/>
+        <child link="multi_camera_rig_mount"/>
         <origin xyz="0.0 0.0 0.0" rpy="${pi/2} 0 0"/>
-    </joint> -->
-    <!-- ROS2_CONTROL -->
-    <!-- HUSKY ros2_control block (binds joints(arg to hardware) -->
-    <!-- <xacro:include filename="$(find husky_xarm6_mcr_description)/urdf/xarm6/xarm6_ros2_control.xacro"/>
-    <xacro:xarm6_ros2_control prefix="$(arg manipulator_prefix)" sim="$(arg sim)"/>
-    <gazebo>
-        <plugin filename="gz_ros2_control-system" name="gz_ros2_control::GazeboSimROS2ControlPlugin">
-            <robot_param>robot_description</robot_param>
-            <robot_param_node>robot_state_publisher</robot_param_node>
-            <parameters>$(find husky_xarm6_mcr_control)/config/controllers.yaml</parameters>
-        </plugin>
-    </gazebo> -->
-    <!-- Gazebo -->
-    <!-- <xacro:include filename="$(find husky_xarm6_mcr_description)/urdf/xarm6/xarm6_gazebo.xacro"/>
-    <xacro:xarm6_gazebo prefix="$(arg manipulator_prefix)"/> -->
+    </joint>
 </robot>

File: husky_xarm6_mcr_description/urdf/xarm6/xarm6_macro.urdf.xacro (robot description, xacro)
@@ -175,5 +175,5 @@
       <dynamics damping="1.0" friction="1.0"/>
     </joint>
-    <!-- Optional EEF stub (commented)
+    <!-- Optional EEF stub -->
     <link name="${prefix}link_eef"/>
     <joint name="${prefix}joint_eef" type="fixed">
@@ -182,5 +182,4 @@
       <child  link="${prefix}link_eef"/>
     </joint>
-    -->
     <!-- Gazebo -->
     <xacro:if value="${use_gazebo}">

File: husky_xarm6_mcr_description/urdf/xarm6/xarm6_ros2_control.xacro (robot description, xacro)
@@ -11,5 +11,7 @@
                     <command_interface name="position"/>
                     <command_interface name="velocity"/>
-                    <state_interface name="position"/>
+                    <state_interface name="position">
+                        <param name="initial_value">${pi/2}</param>
+                    </state_interface>
                     <state_interface name="velocity"/>
                 </joint>
@@ -17,5 +19,7 @@
                     <command_interface name="position"/>
                     <command_interface name="velocity"/>
-                    <state_interface name="position"/>
+                    <state_interface name="position">
+                        <param name="initial_value">-${pi/4}</param>
+                    </state_interface>
                     <state_interface name="velocity"/>
                 </joint>
@@ -23,5 +27,7 @@
                     <command_interface name="position"/>
                     <command_interface name="velocity"/>
-                    <state_interface name="position"/>
+                    <state_interface name="position">
+                        <param name="initial_value">-${pi/4}</param>
+                    </state_interface>
                     <state_interface name="velocity"/>
                 </joint>
@@ -29,5 +35,7 @@
                     <command_interface name="position"/>
                     <command_interface name="velocity"/>
-                    <state_interface name="position"/>
+                    <state_interface name="position">
+                        <param name="initial_value">0.0</param>
+                    </state_interface>
                     <state_interface name="velocity"/>
                 </joint>
@@ -35,5 +43,7 @@
                     <command_interface name="position"/>
                     <command_interface name="velocity"/>
-                    <state_interface name="position"/>
+                    <state_interface name="position">
+                        <param name="initial_value">0.0</param>
+                    </state_interface>
                     <state_interface name="velocity"/>
                 </joint>
@@ -41,5 +51,7 @@
                     <command_interface name="position"/>
                     <command_interface name="velocity"/>
-                    <state_interface name="position"/>
+                    <state_interface name="position">
+                        <param name="initial_value">${pi/2}</param>
+                    </state_interface>
                     <state_interface name="velocity"/>
                 </joint>

Commit message: Implementing image bridge. Fixed bug in multi camera group in srdf file.

File: husky_xarm6_mcr_description/srdf/husky_xarm6_mcr.srdf.xacro (robot description, xacro)
@@ -25,5 +25,5 @@
         <link name="zed2i_camera_center"/>
         <link name="ximea_camera_link"/>
-        <link name="ffs_camera_link"/>
+        <link name="firefly_camera_link"/>
         <link name="multi_camera_rig_link"/>
     </group>

Commit message: began adding in the localization functionality, but commented this out for the moment. Then started trying to get the hardware version functional. Currently I am still trying to get the controllers brought up.

File: husky_xarm6_mcr_description/srdf/husky_xarm6_mcr.srdf.xacro (robot description, xacro)
@@ -5,5 +5,5 @@
     <xacro:arg name="platform_prefix" default="a200_"/>
     <!-- Import multi camera rig SRDF -->
-    <xacro:include filename="$(find multi_cam_rig_description)/srdf/multi_cam_rig.srdf.xacro"/>
+    <xacro:include filename="$(find multi_camera_rig_description)/srdf/multi_cam_rig.srdf.xacro"/>
     <!--GROUPS: Representation of a set of joints and links. This can be useful for specifying DOF to plan for, defining arms, end effectors, etc-->
     <group name="$(arg platform_prefix)platform">

File: husky_xarm6_mcr_description/urdf/husky_xarm6_mcr.urdf.xacro (robot description, xacro)
@@ -2,10 +2,12 @@
 <robot xmlns:xacro="http://ros.org/wiki/xacro" name="husky_xarm6_mcr">
     <!-- Arguments -->
-    <xacro:arg name="sim" default="true"/>
+    <xacro:arg name="use_gazebo" default="false"/>
     <xacro:arg name="manipulator_prefix" default="xarm6_"/>
     <xacro:arg name="platform_prefix" default="a200_"/>
+    <xacro:arg name="robot_ip" default="192.168.1.205"/>
+    <xacro:arg name="report_type" default="normal"/>
     <!-- HUSKY PLATFORM & ATTACHMENTS -->
     <xacro:include filename="$(find husky_xarm6_mcr_description)/urdf/husky/a200_macro.urdf.xacro"/>
-    <xacro:a200 prefix="$(arg platform_prefix)" use_gazebo="$(arg sim)"/>
+    <xacro:a200 prefix="$(arg platform_prefix)" use_gazebo="$(arg use_gazebo)"/>
     <!-- X-RAIL RISER -->
     <xacro:include filename="$(find husky_xarm6_mcr_description)/urdf/risers/x_rail_macro.urdf.xacro"/>
@@ -20,15 +22,17 @@
     <!-- ROS2_CONTROL -->
     <xacro:include filename="$(find husky_xarm6_mcr_description)/urdf/husky/husky_ros2_control.xacro"/>
-    <xacro:husky_ros2_control prefix="$(arg platform_prefix)" use_gazebo="$(arg sim)"/>
+    <xacro:husky_ros2_control prefix="$(arg platform_prefix)" use_gazebo="$(arg use_gazebo)"/>
     <xacro:include filename="$(find husky_xarm6_mcr_description)/urdf/xarm6/xarm6_ros2_control.xacro"/>
-    <xacro:xarm6_ros2_control prefix="$(arg manipulator_prefix)" use_gazebo="$(arg sim)"/>
-    <gazebo>
-        <plugin filename="gz_ros2_control-system" name="gz_ros2_control::GazeboSimROS2ControlPlugin">
-            <parameters>$(find husky_xarm6_mcr_control)/config/controllers.yaml</parameters>
-        </plugin>
-    </gazebo>
+    <xacro:xarm6_ros2_control prefix="$(arg manipulator_prefix)" use_gazebo="$(arg use_gazebo)" robot_ip="$(arg robot_ip)" report_type="$(arg report_type)"/>
+    <xacro:if value="$(arg use_gazebo)">
+        <gazebo>
+            <plugin filename="gz_ros2_control-system" name="gz_ros2_control::GazeboSimROS2ControlPlugin">
+                <parameters>$(find husky_xarm6_mcr_control)/config/controllers.yaml</parameters>
+            </plugin>
+        </gazebo>
+    </xacro:if>
     <!-- MULTI CAMERA RIG -->
-    <xacro:include filename="$(find multi_cam_rig_description)/urdf/multi_cam_rig_macro.urdf.xacro"/>
-    <xacro:multi_camera_rig use_gazebo="$(arg sim)"/>
+    <xacro:include filename="$(find multi_camera_rig_description)/urdf/multi_camera_rig_macro.urdf.xacro"/>
+    <xacro:multi_camera_rig use_gazebo="$(arg use_gazebo)"/>
     <joint name="tool_mount" type="fixed">
         <parent link="$(arg manipulator_prefix)link_eef"/>
@@ -36,3 +40,15 @@
         <origin xyz="0.0 0.0 0.0" rpy="${pi/2} 0 0"/>
     </joint>
+    <!-- SWIFTNAV DURO GPS (mounted on top of base_link) -->
+    <!-- <xacro:property name="name" value="gps"/>
+    <xacro:include filename="$(find husky_xarm6_mcr_description)/urdf/sensors/swiftnav_duro.urdf.xacro"/>
+    <xacro:swiftnav_duro parent_link="$(arg platform_prefix)base_link">
+        <origin xyz="0.0 0.0 0.3" rpy="0 0 0"/>
+    </xacro:swiftnav_duro> -->
+    <!-- MICROSTRAIN IMU (mounted inside base_link) -->
+    <!-- <xacro:property name="name" value="imu"/>
+    <xacro:include filename="$(find husky_xarm6_mcr_description)/urdf/sensors/microstrain_imu.urdf.xacro"/>
+    <xacro:microstrain_imu parent_link="$(arg platform_prefix)base_link" update_rate="100">
+        <origin xyz="0.0 0.0 0.05" rpy="0 0 0"/>
+    </xacro:microstrain_imu> -->
 </robot>

File: husky_xarm6_mcr_description/urdf/xarm6/xarm6_ros2_control.xacro (robot description, xacro)
@@ -1,5 +1,5 @@
 <?xml version="1.0"?>
 <robot xmlns:xacro="http://ros.org/wiki/xacro">
-    <xacro:macro name="xarm6_ros2_control" params="prefix use_gazebo:=true">
+    <xacro:macro name="xarm6_ros2_control" params="prefix use_gazebo:=true hw_ns:='xarm' velocity_control:='false' robot_ip:='192.168.1.205' report_type:='normal' baud_checkset:='true'">
         <xacro:if value="${use_gazebo}">
             <ros2_control name="${prefix}gazebo_system" type="system">
@@ -58,16 +58,39 @@
             </ros2_control>
         </xacro:if>
-        <!-- Real hardware (later) -->
-        <!-- <xacro:unless value="${use_gazebo}">
-            <ros2_control name="${prefix}uf_hw" type="system">
+        <!-- Real hardware -->
+        <xacro:unless value="${use_gazebo}">
+            <xacro:include filename="$(find xarm_description)/urdf/xarm6/xarm6.ros2_control.xacro" />
+            <xacro:include filename="$(find xarm_description)/urdf/xarm6/xarm6.transmission.xacro" />
+            <xacro:xarm6_ros2_control prefix="${prefix}"
+                velocity_control="${velocity_control}"
+                ros2_control_plugin="uf_robot_hardware/UFRobotSystemHardware"
+                hw_ns="${hw_ns}" add_gripper="false" add_bio_gripper="false"
+                robot_ip="${robot_ip}" report_type="${report_type}"
+                baud_checkset="${baud_checkset}" default_gripper_baud="2000000"
+                joint1_lower_limit="${-pi*0.99}" joint1_upper_limit="${pi*0.99}"
+                joint2_lower_limit="${-2.059}" joint2_upper_limit="${2.0944}"
+                joint3_lower_limit="${-pi*0.99}" joint3_upper_limit="${0.19198}"
+                joint4_lower_limit="${-pi*0.99}" joint4_upper_limit="${pi*0.99}"
+                joint5_lower_limit="${-1.69297}" joint5_upper_limit="${pi*0.99}"
+                joint6_lower_limit="${-pi*0.99}" joint6_upper_limit="${pi*0.99}"
+            />
+            <xacro:xarm6_transmission prefix="${prefix}" hard_interface="EffortJointInterface" reduction="100"/>
+            <!-- <ros2_control name="${prefix}uf_robot_hardware/UFRobotSystemHardware" type="system">
                 <hardware>
                     <plugin>uf_robot_hardware/UFRobotSystemHardware</plugin>
-                    <param name="hw_ns">${prefix}xarm</param>
+                    <param name="hw_ns">${prefix}${hw_ns}</param>
+                    <param name="velocity_control">${velocity_control}</param>
+                    <param name="prefix">P${prefix}</param>
+                    <param name="robot_ip">R${robot_ip}</param>
+                    <param name="report_type">${report_type}</param>
                     <param name="dof">6</param>
+                    <param name="baud_checkset">${baud_checkset}</param>
+                    <param name="default_gripper_baud">${default_gripper_baud}</param>
                     <param name="robot_type">xarm</param>
-                    <param name="velocity_control">false</param>
+                    <param name="add_gripper">${add_gripper}</param>
                 </hardware>
                 <joint name="${prefix}joint1">
                     <command_interface name="position"/>
+                    <command_interface name="velocity"/>
                     <state_interface name="position"/>
                     <state_interface name="velocity"/>
@@ -75,4 +98,5 @@
                 <joint name="${prefix}joint2">
                     <command_interface name="position"/>
+                    <command_interface name="velocity"/>
                     <state_interface name="position"/>
                     <state_interface name="velocity"/>
@@ -80,4 +104,5 @@
                 <joint name="${prefix}joint3">
                     <command_interface name="position"/>
+                    <command_interface name="velocity"/>
                     <state_interface name="position"/>
                     <state_interface name="velocity"/>
@@ -85,4 +110,5 @@
                 <joint name="${prefix}joint4">
                     <command_interface name="position"/>
+                    <command_interface name="velocity"/>
                     <state_interface name="position"/>
                     <state_interface name="velocity"/>
@@ -90,4 +116,5 @@
                 <joint name="${prefix}joint5">
                     <command_interface name="position"/>
+                    <command_interface name="velocity"/>
                     <state_interface name="position"/>
                     <state_interface name="velocity"/>
@@ -95,9 +122,10 @@
                 <joint name="${prefix}joint6">
                     <command_interface name="position"/>
+                    <command_interface name="velocity"/>
                     <state_interface name="position"/>
                     <state_interface name="velocity"/>
                 </joint>
-            </ros2_control>
-        </xacro:unless> -->
+            </ros2_control> -->
+        </xacro:unless>
     </xacro:macro>
 </robot>
