Commit message: updated the collision for the xrail riser, gave additional padding for the batter mounts and laptop ledge.

File: husky_xarm6_mcr_description/urdf/risers/x_rail_macro.urdf.xacro (robot description, xacro)
@@ -5,4 +5,7 @@
         <!-- Build namespace prefix -->
         <xacro:property name="ns_prefix" value="${namespace}/${prefix}"/>
+        <xacro:property name="height" value="0.33" />
+        <xacro:property name="width" value="0.46" />
+        <xacro:property name="depth" value="1.1" />
         <!-- X-Rail Riser Link -->
         <link name="${ns_prefix}x_rail_riser_link">
@@ -15,8 +18,7 @@
             </visual>
             <collision>
-                <origin xyz="0 0 0" rpy="0 0 0"/>
+                <origin xyz="0 0 ${height/2}" rpy="0 0 0"/>
                 <geometry>
-                    <!-- <mesh filename="package://husky_xarm6_mcr_description/meshes/x_rail_riser_collision.stl" scale="1 1 1"/> -->
-                    <mesh filename="file://$(find husky_xarm6_mcr_description)/meshes/x_rail_riser_collision.stl"/>
+                    <box size="${width} ${depth} ${height}"/>
                 </geometry>
             </collision>

Commit message: updated collision xrail model.

File: husky_xarm6_mcr_description/urdf/risers/x_rail_macro.urdf.xacro (robot description, xacro)
@@ -14,5 +14,5 @@
         <xacro:property name="riser_y_origin" value="-0.078" />
         <xacro:property name="riser_z_origin" value="0" />
-        <xacro:property name="riser_y_offset" value="0.125" />
+        <xacro:property name="riser_y_offset" value="-0.125" />
         <xacro:property name="riser_z_offset" value="-0.02" />
         <!-- Battery Size -->

Commit message: Added additional padding to the riser collision model.

File: husky_xarm6_mcr_description/urdf/risers/x_rail_macro.urdf.xacro (robot description, xacro)
@@ -33,5 +33,5 @@
                 <origin xyz="${riser_x_origin} ${riser_y_offset} ${riser_z_origin + riser_z_offset + riser_z_size/2}" rpy="0 0 0"/>
                 <geometry>
-                    <box size="${riser_x_size} ${riser_y_size + riser_y_extension} ${riser_z_size}"/>
+                    <box size="${riser_x_size + 0.02} ${riser_y_size + riser_y_extension + 0.02} ${riser_z_size + 0.02}"/>
                 </geometry>
             </collision>
@@ -40,5 +40,5 @@
                 <origin xyz="0 0 ${battery_z_origin}" rpy="0 0 0"/>
                 <geometry>
-                    <box size="${riser_x_size} ${riser_y_size} ${battery_z_size}"/>
+                    <box size="${riser_x_size + 0.02} ${riser_y_size + 0.02} ${battery_z_size + 0.02}"/>
                 </geometry>
             </collision>
